File: Laser_Driver_v3/laser_driver_v3.kicad_pcb (KiCad board)
At the start: 2 copper layers, 300 x 200 mm, 312 parts, among them J1 SMA Isolated Coax, J2 SMA Isolated Coax, J3 10MHz Ref SMA, J4 +/-15V PWR, J5 +5V Laser, J6 3V3 Teensy, J7 ADC Teensy, J8 TEC H-bridge leads, Q1 IRF540NPBF, Q10 IRF9540N, Q11 IRLB8721PBF, Q12 IRF9540N, Q13 IRLB8721PBF, Q14 IRF9540N, Q15 IRLML6344TRPBF, Q16 IRLML6344TRPBF, Q2 IRF9540NPBF, Q3 IRF540NPBF, Q4 IRF9540NPBF, Q5 Q_NPN MJL21193, Q6 Q_PNP_MJL21194, Q7 IRLB8721PBF, Q8 IRF9540N, Q9 IRLB8721PBF, T1 Talema_6202W_30VA_2x18VAC, U1 MC7808CTG, U10 LT3042EMSE +14.3V, U11 LT3094EMSE -14.3V, U12 LM4040DBZ-6.2, U13 LM4040DBZ-6.2, U14 MC7812CTG, U15 MC7808CTG, U16 LT3045EMSE 5V, U17 LT3045EMSE 5V, U18 OPA192IDR, U19 OPA192IDR, U2 LT3042EMSE +5.5V, U20 OPA192IDR, U21 OPA551U, U22 OPA551U, U23 OPA192IDR, U24 OPA192IDR, U25 INA826, U26 INA826, U27 INA826, U28 INA826, U29 OPA2141AID, U3 LTC6655BHLS8-5, U30 74AHCT125, U31 AD9833xRM, U32 AD5064BRUZ, U33 AD9833xRM, U34 LMV7219M5, U35 SN74LVC1G3157DBVR, U36 CDCE913PWG4, U4 OPA192IDR, U5 MC7812CTG, U6 MC7805CTG, U7 LT3045EMSE 3.3V, U8 LP5907MFX-1.8, U9 TPS7A39DGNR, Y1 ASE-10.000MHZ-LC-T

Commit message: Clearing ERC errors. laying out components.
Parts:
- removed R90, R91, R92, R93, R94, R95, R96: 47R prot, Resistor_SMD:R_0402_1005Metric
- J3: footprint Connector_Coaxial:BNC_Win_364A2x95_Horizontal -> Connector_Coaxial:SMA_BAT_Wireless_BWSMA-KWE-Z001
- U35: footprint Package_TO_SOT_SMD:SOT-23-5 -> Package_TO_SOT_SMD:SOT-23-6_Handsoldering
- moved R104 75.6 mm to (352.5, 137.0), turned to -90 degrees
- moved R80 75.4 mm to (337.0, 186.8), turned to 90 degrees
- moved D7 73.0 mm to (151.4, 197.0)
- moved R106 68.4 mm to (347.5, 137.0), turned to 90 degrees
- moved R108 65.7 mm to (340.0, 137.0), turned to -90 degrees
- moved C70 64.3 mm to (335.6, 183.0), turned to 180 degrees
- moved C69 62.6 mm to (330.4, 185.5), turned to 180 degrees
- moved R105 57.8 mm to (352.5, 124.5), turned to -90 degrees
- moved A1 56.3 mm to (346.6, 215.2), turned to 90 degrees
- moved R107 56.0 mm to (342.5, 124.5), turned to 90 degrees
- moved R117 55.8 mm to (337.5, 99.0), turned to 90 degrees
- moved R114 54.7 mm to (342.5, 99.5), turned to 90 degrees
- moved R84 54.2 mm to (331.5, 181.3), turned to 90 degrees
- moved R83 51.9 mm to (324.6, 185.5), turned to 180 degrees
- moved R115 48.7 mm to (340.0, 111.5), turned to 90 degrees
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Connections:
- Q13 pad 2: unconnected-(Q13-D-Pad2) -> +6V_TEC
- Q14 pad 3: unconnected-(Q14-S-Pad3) -> -6V_TEC
- R_NTC1 pad 1: unconnected-(R_NTC1-Pad1) -> 3V3
- R_NTC2 pad 1: unconnected-(R_NTC2-Pad1) -> 3V3
- U36 pad 6: Net-(U36-VDDOUT-Pad6) -> 3V3
- U36 pad 7: Net-(U36-VDDOUT-Pad6) -> 3V3
Other:
- board size 300 x 200 mm -> 306.2 x 200 mm

Commit message: Update to teensy pinout and config. Working on PCB
Improved pin selection on Teensy for better operation.
Started working through the PCB from in the power input.
Updating footprints and getting the layout organized.
Parts:
- added U38: CR2013-MI2120, Display:CR2013-MI2120, F.Cu at (378.6, 175.2)
- C1, C2, C7, C8, R2, R3, R7: moved to B.Cu
- C62, C63: footprint Capacitor_SMD:C_1210_3225Metric -> Capacitor_SMD:C_1206_3216Metric_Pad1.33x1.80mm_HandSolder
- D1: footprint Diode_SMD:Diode_Bridge_Diotec_ABS -> Diode_THT:Diode_Bridge_Vishay_GBU
- J4: value +/-15V PWR -> Screw_Terminal_01x03; footprint Connector_PinHeader_2.54mm:PinHeader_1x02_P2.54mm_Vertical -> TerminalBlock_RND:TerminalBlock_RND_205-00233_1x03_P5.08mm_Horizontal
- R1, R4, R5, R6: footprint Resistor_SMD:R_0402_1005Metric -> Resistor_SMD:R_0805_2012Metric_Pad1.20x1.40mm_HandSolder; moved to B.Cu
- R8, R9: footprint Resistor_SMD:R_0402_1005Metric -> Resistor_SMD:R_2512_6332Metric_Pad1.40x3.35mm_HandSolder; moved to B.Cu
- T1: value Talema_6202W_30VA_2x18VAC -> Talema_70064k_25VA_2x18VAC; footprint Connector_PinHeader_2.54mm:PinHeader_1x04_P2.54mm_Vertical -> Talema7006x:XFMR_70060K
- U10, U2: footprint Package_DFN_QFN:DFN-10-1EP_3x3mm_P0.5mm_EP1.65x2.38mm -> Package_SO:MSOP-10-1EP_3x3mm_P0.5mm_EP2.2x3.1mm_Mask1.83x1.89mm_ThermalVias
- U11: footprint Package_SO:MSOP-10_3x3mm_P0.5mm -> Package_SO:Analog_MSOP-12-16-1EP_3x4.039mm_P0.5mm_EP1.651x2.845mm_ThermalVias
- U16, U17, U7: footprint Package_DFN_QFN:DFN-10-1EP_3x3mm_P0.5mm_EP1.65x2.38mm -> Package_SO:Analog_MSOP-12-16-1EP_3x4.039mm_P0.5mm_EP1.651x2.845mm_ThermalVias
- moved J8 147.0 mm to (20.5, 54.7)
- moved J4 107.2 mm to (56.0, 147.2)
- moved T1 104.0 mm to (81.5, 189.0)
- moved D4 89.9 mm to (36.1, 73.5)
- moved F1 88.2 mm to (57.5, 156.2), turned to -90 degrees
- moved D7 88.0 mm to (150.5, 109.0)
- moved R2 85.8 mm to (87.2, 147.8)
- moved R3 82.8 mm to (69.7, 147.8), turned to 180 degrees
- moved R4 81.0 mm to (95.5, 143.8), turned to -90 degrees
- moved R1 79.7 mm to (80.0, 141.8), turned to 90 degrees
- moved C1 74.0 mm to (87.7, 140.8), turned to 180 degrees
- moved R5 73.2 mm to (69.5, 137.0)
- moved Q1 70.8 mm to (89.0, 145.0)
- moved R6 70.3 mm to (90.2, 136.8), turned to 180 degrees
- moved C2 70.1 mm to (69.4, 141.2)
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Connections:
- A1 pad D10: unconnected-(A1-(CS)D10-PadD10) -> CS_3V3
- A1 pad D12: unconnected-(A1-(SDI)D12-PadD12) -> MISO_3V3
- A1 pad D2: CS_3V3 -> DDS1_FSYNC
- A1 pad D26: unconnected-(A1-A12-PadD26) -> TFT_MOSI
- A1 pad D27: unconnected-(A1-A13-PadD27) -> TFT_SCK
- A1 pad D28: unconnected-(A1-PadD28) -> Net-(U38-~{CS})
- A1 pad D29: unconnected-(A1-PadD29) -> Net-(U38-D/~{C})
- A1 pad D3: DDS1_FSYNC -> DDS2_FSYNC
- A1 pad D30: unconnected-(A1-PadD30) -> Net-(U38-RESET)
- A1 pad D4: DDS2_FSYNC -> DDS1_RESET
- A1 pad D5: unconnected-(A1-PadD5) -> DDS2_RESET
- A1 pad D7: unconnected-(A1-PadD7) -> AD5064_CLR
- D1 pad 2: Net-(D1--) -> Net-(D1-Pad2)
- D1 pad 3: Net-(T1-SA) -> Net-(D1-Pad3)
- D1 pad 4: Net-(T1-SB) -> Net-(D1--)
- F1 pad 2: Net-(T1-AA) -> Net-(F1-Pad2)
- J4 pad 1: (no net) -> Earth
- J4 pad 2: (no net) -> 0Vac
- T1 pad 3: Net-(T1-SA) -> 0Vac
- T1 pad 4: unconnected-(T1-SC-Pad4) -> Net-(F1-Pad2)

Commit message: Working through power supply layout and footprints
Parts:
- C10, C9, R14: moved to B.Cu
- D12, D13, D4, D5, D6: footprint Diode_THT:D_DO-41_SOD81_P10.16mm_Horizontal -> Diode_THT:D_DO-15_P12.70mm_Horizontal
- U16, U17: footprint Package_SO:Analog_MSOP-12-16-1EP_3x4.039mm_P0.5mm_EP1.651x2.845mm_ThermalVias -> Package_SO:MSOP-12-1EP_3x4.039mm_P0.65mm_EP1.651x2.845mm_ThermalVias
- U3: footprint Package_SO:SOIC-8_3.9x4.9mm_P1.27mm -> Package_SO:MSOP-8_3x3mm_P0.65mm
- moved D4 99.2 mm to (125.8, 31.0)
- moved U38 90.6 mm to (291.7, 149.5), turned to -90 degrees
- moved C41 65.4 mm to (169.5, 168.0)
- moved C42 44.2 mm to (175.5, 192.5)
- moved C38 30.0 mm to (128.9, 149.0)
- moved R32 29.7 mm to (142.2, 154.2)
- moved C51 28.1 mm to (204.0, 39.1), turned to -90 degrees
- moved C52 27.3 mm to (206.0, 39.1), turned to -90 degrees
- moved D12 27.1 mm to (196.0, 31.0)
- moved C49 25.7 mm to (191.5, 39.1), turned to -90 degrees
- moved C50 24.9 mm to (193.5, 39.1), turned to -90 degrees
- moved R34 24.2 mm to (219.0, 38.2)
- moved R10 23.7 mm to (149.0, 41.2), turned to -90 degrees
- moved D5 23.5 mm to (267.8, 33.5)
- moved C54 23.1 mm to (224.0, 40.2), turned to -90 degrees
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Connections:
- C55 pad 1: 5VLaser -> Net-(U17-OUTS)
- C56 pad 1: -6V_TEC -> Net-(U16-SET)
- C57 pad 1: 5VLaser -> Net-(U16-OUTS)
- R35 pad 1: Net-(U16-SET) -> Net-(U17-OUTS)
- R35 pad 2: -6V_TEC -> 5VLaser
- R36 pad 1: Net-(U17-SET) -> Net-(U16-OUTS)
- R36 pad 2: -6V_TEC -> 5VLaser
- R37 pad 1: -6V_TEC -> Net-(U16-SET)
- U16 pad 10: 5VLaser -> Net-(U16-OUTS)
- U16 pad 11: (no net) -> Net-(U16-OUTS)
- U16 pad 12: (no net) -> Net-(U16-OUTS)
- U16 pad 5: -6V_TEC -> unconnected-(U16-PG-Pad5)
- U16 pad 6: Net-(U16-EN/UV) -> -6V_TEC
- U16 pad 7: Net-(U16-SET) -> Net-(U16-EN/UV)
- U16 pad 8: -6V_TEC -> Net-(U16-SET)
- U16 pad 9: 5VLaser -> -6V_TEC
- U17 pad 10: 5VLaser -> Net-(U17-OUTS)
- U17 pad 11: (no net) -> Net-(U17-OUTS)
- U17 pad 12: (no net) -> Net-(U17-OUTS)
- U17 pad 5: -6V_TEC -> unconnected-(U17-PG-Pad5)
- U17 pad 6: Net-(U16-EN/UV) -> -6V_TEC
- U17 pad 7: Net-(U17-SET) -> Net-(U16-EN/UV)
- U17 pad 8: -6V_TEC -> Net-(U16-SET)
- U17 pad 9: 5VLaser -> -6V_TEC

Commit message: Began routing.
Parts:
- R1: moved to F.Cu
- moved D7 21.1 mm to (131.1, 100.8)
- moved C1 14.5 mm to (88.4, 126.2)
- moved C2 14.5 mm to (70.2, 126.8)
- moved C3 14.5 mm to (92.0, 108.2)
- moved C4 14.5 mm to (72.2, 108.2)
- moved C5 14.5 mm to (92.0, 87.2)
- moved C6 14.5 mm to (72.5, 87.2)
- moved C7 14.5 mm to (84.2, 121.0)
- moved C8 14.5 mm to (77.5, 121.0)
- moved Q1 14.5 mm to (89.8, 130.5)
- moved Q2 14.5 mm to (68.7, 130.5)
- moved R2 14.5 mm to (88.0, 133.2)
- moved R3 14.5 mm to (70.5, 133.2)
- moved R4 14.5 mm to (96.2, 129.2)
- moved R5 14.5 mm to (70.2, 122.5)
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Connections:
- net Net-(D1-+) renamed /Mains to +-18V/+23V
- net Net-(D1--) renamed /Mains to +-18V/-23V
- net Net-(D1-Pad2) renamed /Mains to +-18V/+18Vac
- net Net-(D2-K) renamed /Mains to +-18V/-18VNF
- net Net-(D3-A) renamed /Mains to +-18V/+18VNF
- D1 pad 3: Net-(D1-Pad3) -> -18V
- T1 pad 14: Net-(D1-Pad3) -> -18V
Routing:
- net -6V_TEC: track 0.00 -> 110.0 mm
- net 0Vac: track 0.00 -> 84.3 mm
- net -18V: track 0.00 -> 83.2 mm
- net /Mains to +-18V/+18Vac: track 0.00 -> 81.5 mm
- net Net-(F1-Pad2): track 0.00 -> 74.2 mm
- net /Mains to +-18V/-18VNF: track 0.00 -> 28.5 mm
- net 120Vac: track 0.00 -> 23.0 mm
- net /Mains to +-18V/-23V: track 0.00 -> 18.1 mm
- net /Mains to +-18V/+23V: track 0.00 -> 17.9 mm
- net /Mains to +-18V/+18VNF: track 0.00 -> 13.0 mm
- net Net-(D2-A): track 0.00 -> 10.5 mm
- net Earth: track 0.00 -> 8.07 mm
- net +18V: track 0.00 -> 4.60 mm
