File: Laser_Driver_v3/Mains_to_pm18V.kicad_sch (KiCad schematic)
At the start: 27 parts, among them J1 Screw_Terminal_01x03, Q1 IRF540NPBF, Q2 IRF9540NPBF, T1 Talema 62064, T2 Talema 62081

Commit message: Changed xfrmers, paralled BJTs for cap multiplier
Changed the transformers to more appropriate voltages.
Made the BJTs for the cap multipliers in parallel to better handle the load.
Simulated the output ripple for the 6V.
Clarifying notes, removed LT1028 changed to OPA192 to match circuit as drawn.
Changed divider values for the TEC_zero value to be 1.2 V as designed.
Parts:
- T1: value Talema 62064 -> Talema 62063
Connections:
- net +18Vac: no longer names the net of D1.2, T1.Blue (-9V)
- net +23V: no longer names the net of D1.1 (+), Q1.1 (D), R2.1
- net -18Vac: no longer names the net of D1.3, T1.Green (+9V)
- net -23V: no longer names the net of D1.4 (-), Q2.1 (D), R3.1
Changed lines of the file:
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@@
-		)
-	)
-	(label "-23V"
-		(at 118.11 82.55 0)
-		(effects
-			(font
-				(size 1.27 1.27)
-			)
-			(justify left bottom)
-		)
-	)
-	(label "-18Vac"
-		(at 99.06 78.74 0)
-		(effects
-			(font
-				(size 1.27 1.27)
-			)
-			(justify left bottom)
-		)
-	)
-	(label "+23V"
-		(at 123.19 52.07 0)
-		(effects
-			(font
-				(size 1.27 1.27)
-			)
-			(justify left bottom)
-		)
-	)
-	(label "+18Vac"
-		(at 106.68 53.34 0)
-		(effects
-			(font
-				(size 1.27 1.27)
-			)
-			(justify left bottom)
 		)
 	)
@@
 			)
 		)
-		(property "Value" "Talema 62064"
+		(property "Value" "Talema 62063"
 			(at 78.74 55.88 0)
 			(show_name no)
@@
 		(dnp no)
 		(property "Reference" "F1"
-			(at 49.784 55.118 90)
+			(at 49.784 56.134 90)
 			(show_name no)
 			(do_not_autoplace no)
@@
 		)
 		(property "Value" "1A SlowBlow"
-			(at 49.53 56.642 90)
+			(at 49.53 60.706 90)
 			(show_name no)
 			(do_not_autoplace no)
@@
 		(in_pos_files yes)
 		(dnp no)
-		(fields_autoplaced yes)
 		(property "Reference" "TH1"
-			(at 60.0075 52.07 90)
+			(at 59.436 56.134 90)
 			(show_name no)
 			(do_not_autoplace no)
@@
 		)
 		(property "Value" "Ametherm SL22 10005"
-			(at 60.0075 54.61 90)
-			(show_name no)
-			(do_not_autoplace no)
+			(at 65.024 54.356 90)
+			(show_name no)
+			(do_not_autoplace no)
