File: Laser_Driver_v3/Readback.kicad_sch (KiCad schematic)
At the start: 43 parts, among them J3 10 MHz Isolated Coax, J4 10 MHz Isolated Coax, U25 INA826, U27 INA826, U28 INA826, U29 INA826, U36 OPA2141

Commit message: Renumbered schematics, corrections, power verified
Parts:
- R74: renamed from R81; value 4.53k -> 487R
- R75: renamed from R82; value 4.53k -> 487R
- R78: renamed from R65; value 5.489k -> 8.06k
- R79: renamed from R67; value 5.489k -> 8.06k
- renumbered C_aaf1a2 to C_aaf1a1, C_aaf1a1 to C_aaf1a2, C_aaf1b2 to C_aaf1b1, C_aaf1b1 to C_aaf1b2, C_ef2 to C_ef1, C_ef1 to C_ef2, C_f4 to C_f3, C_f3 to C_f4, J4 to J1, J3 to J2, R91 to R76, R1 to R77, R_aaf1a2 to R_aaf1a1, R_aaf1a1 to R_aaf1a2, R_aaf1b2 to R_aaf1b1, R_aaf1b1 to R_aaf1b2, R_bias3 to R_bias1, R_bias4 to R_bias2, R_f4 to R_f3, R_f3 to R_f4, U28 to U25, U29 to U26, U25 to U27, U27 to U28, U36 to U29, U_TIA8 to U_TIA1, U_TIA6 to U_TIA2, U_TIA4 to U_TIA3, U_TIA1 to U_TIA4, U_TIA2 to U_TIA5, U_TIA5 to U_TIA6
Connections:
- net TEC1_SENSE_N: no longer U28.1 (-)
- net TEC1_SENSE_P: no longer U28.4 (+)
- new net TEC2_SENSE_N: U28.1 (-)
- new net TEC2_SENSE_P: U28.4 (+)
Other:
- note added: "Ext PD TIA: OPA380 Rf=2.7k Bw=1.3MHz | AAF: OPA2141 2-pole 30kHz Butterworth | Teensy ADC1/ADC2 @100kHz DMA lock-in"
- note added: "INA826 gains: Laser G=106 (Rg=487, Vmax=3.0V@600mA) TEC G=7.2 (Rg=8.06k, Vmax=3.0V@2.5A)"
- note added: "READBACK + LOCK-IN SIGNAL PATH | 4x INA826 InAmp | NTC dividers | OPA380 TIA | OPA2141"
- note removed: "Ext PD TIA: OPA380 Rf=2.7k Bw=1.3MHz | AAF: OPA2134 2-pole 30kHz Butterworth | Teensy ADC1/ADC2 @100kHz DMA lock-in"
- note removed: "INA826 gains: Laser G=12 (Rg=4.53k, Vmax=3.0V@600mA) TEC G=20 (Rg=2.61k, Vmax=3.0V@2.5A)"
- note removed: "READBACK + LOCK-IN SIGNAL PATH | 4x INA826 InAmp | NTC dividers | OPA380 TIA | OPA2134 AAF"

Commit message: Update names, footprints, values, and created BOM
Updated files names, foot prints, component values, parts.
Assigned values from Digikey catalog.
Created CSV BOMs for each schematic.
Including a Power analysis now for all components.
Parts:
- C_NTC1, C_NTC2, C_aaf1a1, C_aaf1a2, C_aaf1b1, C_aaf1b2: footprint Capacitor_SMD:C_0402_1005Metric -> Capacitor_SMD:C_0805_2012Metric_Pad1.18x1.45mm_HandSolder
- J1, J2: value 10 MHz Isolated Coax -> SMA Isolated Coax; footprint Connector_Coaxial:BNC_Win_364A2x95_Horizontal -> Connector_Coaxial:SMA_THT_Horizontal
- R74, R75, R76, R77, R78, R79, R_aaf1a1, R_aaf1a2, R_aaf1b1, R_aaf1b2, R_bias1, R_bias2, R_f1, R_f2, R_f3, R_f4: footprint Resistor_SMD:R_0402_1005Metric -> Resistor_SMD:R_0805_2012Metric_Pad1.20x1.40mm_HandSolder
- U29: value OPA2141 -> OPA2141AID; footprint (none) -> Package_SO:SOIC-8_3.9x4.9mm_P1.27mm
Changed lines of the file:
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@@
 			)
 		)
-		(property "Value" "OPA2141"
+		(property "Value" "OPA2141AID"
 			(at 141.478 153.162 0)
 			(show_name no)
@@
 			)
 		)
-		(property "Footprint" ""
+		(property "Footprint" "Package_SO:SOIC-8_3.9x4.9mm_P1.27mm"
 			(at 139.7 165.1 0)
 			(hide yes)
@@
 			)
 		)
-		(property "Footprint" "Capacitor_SMD:C_0402_1005Metric"
+		(property "Footprint" "Capacitor_SMD:C_0805_2012Metric_Pad1.18x1.45mm_HandSolder"
 			(at 190.5 54.61 0)
 			(hide yes)
@@
 			)
 		)
-		(property "Footprint" "Capacitor_SMD:C_0402_1005Metric"
+		(property "Footprint" "Capacitor_SMD:C_0805_2012Metric_Pad1.18x1.45mm_HandSolder"
 			(at 86.36 190.5 0)
 			(hide yes)
@@
 			)
 		)
-		(property "Footprint" "Capacitor_SMD:C_0402_1005Metric"
+		(property "Footprint" "Capacitor_SMD:C_0805_2012Metric_Pad1.18x1.45mm_HandSolder"
 			(at 101.6 187.96 0)
 			(hide yes)
@@
 			)
 		)
-		(property "Footprint" "Resistor_SMD:R_0402_1005Metric"
+		(property "Footprint" "Resistor_SMD:R_0805_2012Metric_Pad1.20x1.40mm_HandSolder"
 			(at 55.88 171.45 0)
 			(hide yes)
@@
 			)
 		)
-		(property "Footprint" "Resistor_SMD:R_0402_1005Metric"
+		(property "Footprint" "Resistor_SMD:R_0805_2012Metric_Pad1.20x1.40mm_HandSolder"
 			(at 203.2 119.38 0)
 			(hide yes)
@@
 			)
 		)
-		(property "Value" "10 MHz Isolated Coax"
+		(property "Value" "SMA Isolated Coax"
 			(at 42.418 140.716 0)
 			(show_name no)
@@
 			)
 		)
-		(property "Footprint" "Connector_Coaxial:BNC_Win_364A2x95_Horizontal"
+		(property "Footprint" "Connector_Coaxial:SMA_THT_Horizontal"
 			(at 34.29 144.78 0)
 			(hide yes)
@@
 			)
 		)
-		(property "Footprint" "Capacitor_SMD:C_0402_1005Metric"
+		(property "Footprint" "Capacitor_SMD:C_0805_2012Metric_Pad1.18x1.45mm_HandSolder"
 			(at 190.5 85.09 0)
 			(hide yes)
@@
 			)
 		)
-		(property "Footprint" "Resistor_SMD:R_0402_1005Metric"
+		(property "Footprint" "Resistor_SMD:R_0805_2012Metric_Pad1.20x1.40mm_HandSolder"
 			(at 115.57 73.66 0)
 			(hide yes)
@@
 			)
 		)
-		(property "Footprint" "Resistor_SMD:R_0402_1005Metric"
+		(property "Footprint" "Resistor_SMD:R_0805_2012Metric_Pad1.20x1.40mm_HandSolder"
 			(at -12.51 279.85 0)
 			(hide yes)
@@
 			)
 		)
-		(property "Footprint" "Resistor_SMD:R_0402_1005Metric"
+		(property "Footprint" "Resistor_SMD:R_0805_2012Metric_Pad1.20x1.40mm_HandSolder"
 			(at -12.51 249.37 0)
 			(hide yes)
@@
 			)
 		)
-		(property "Footprint" "Resistor_SMD:R_0402_1005Metric"
+		(property "Footprint" "Resistor_SMD:R_0805_2012Metric_Pad1.20x1.40mm_HandSolder"
 			(at 31.52 -216.9 0)
 			(hide yes)
@@
 			)
 		)
-		(property "Footprint" "Resistor_SMD:R_0402_1005Metric"
+		(property "Footprint" "Resistor_SMD:R_0805_2012Metric_Pad1.20x1.40mm_HandSolder"
 			(at 92.71 143.51 0)
 			(hide yes)
@@
 			)
 		)
-		(property "Footprint" "Resistor_SMD:R_0402_1005Metric"
+		(property "Footprint" "Resistor_SMD:R_0805_2012Metric_Pad1.20x1.40mm_HandSolder"
 			(at 39.37 69.85 0)
 			(hide yes)
@@
 			)
 		)
-		(property "Footprint" "Capacitor_SMD:C_0402_1005Metric"
+		(property "Footprint" "Capacitor_SMD:C_0805_2012Metric_Pad1.18x1.45mm_HandSolder"
 			(at 102.87 148.59 0)
 			(hide yes)
@@
 			)
 		)
-		(property "Footprint" "Resistor_SMD:R_0402_1005Metric"
+		(property "Footprint" "Resistor_SMD:R_0805_2012Metric_Pad1.20x1.40mm_HandSolder"
 			(at 82.55 143.51 0)
 			(hide yes)
@@
 			)
 		)
-		(property "Footprint" "Resistor_SMD:R_0402_1005Metric"
+		(property "Footprint" "Resistor_SMD:R_0805_2012Metric_Pad1.20x1.40mm_HandSolder"
 			(at 57.15 132.08 0)
 			(hide yes)
@@
 			)
 		)
-		(property "Value" "10 MHz Isolated Coax"
+		(property "Value" "SMA Isolated Coax"
 			(at 41.148 180.086 0)
 			(show_name no)
@@
 			)
 		)
-		(property "Footprint" "Connector_Coaxial:BNC_Win_364A2x95_Horizontal"
+		(property "Footprint" "Connector_Coaxial:SMA_THT_Horizontal"
 			(at 33.02 184.15 0)
 			(hide yes)
@@
 			)
 		)
-		(property "Footprint" "Resistor_SMD:R_0402_1005Metric"
+		(property "Footprint" "Resistor_SMD:R_0805_2012Metric_Pad1.20x1.40mm_HandSolder"
 			(at 81.28 182.88 0)
 			(hide yes)
@@
 			)
 		)
-		(property "Footprint" "Resistor_SMD:R_0402_1005Metric"
+		(property "Footprint" "Resistor_SMD:R_0805_2012Metric_Pad1.20x1.40mm_HandSolder"
 			(at 91.44 182.88 0)
 			(hide yes)
@@
 			)
 		)
-		(property "Footprint" "Resistor_SMD:R_0402_1005Metric"
+		(property "Footprint" "Resistor_SMD:R_0805_2012Metric_Pad1.20x1.40mm_HandSolder"
 			(at 114.3 41.91 0)
 			(hide yes)
@@
 			)
 		)
-		(property "Footprint" "Resistor_SMD:R_0402_1005Metric"
+		(property "Footprint" "Resistor_SMD:R_0805_2012Metric_Pad1.20x1.40mm_HandSolder"
 			(at 31.52 -186.42 0)
 			(hide yes)
@@
 			)
 		)
-		(property "Footprint" "Resistor_SMD:R_0402_1005Metric"
+		(property "Footprint" "Resistor_SMD:R_0805_2012Metric_Pad1.20x1.40mm_HandSolder"
 			(at 39.37 41.91 0)
 			(hide yes)
@@
 			)
 		)
-		(property "Footprint" "Resistor_SMD:R_0402_1005Metric"
+		(property "Footprint" "Resistor_SMD:R_0805_2012Metric_Pad1.20x1.40mm_HandSolder"
 			(at 250.19 118.11 0)
 			(hide yes)
@@
 			)
 		)
-		(property "Footprint" "Capacitor_SMD:C_0402_1005Metric"
+		(property "Footprint" "Capacitor_SMD:C_0805_2012Metric_Pad1.18x1.45mm_HandSolder"
 			(at 87.63 151.13 0)
 			(hide yes)

Commit message: Clearing ERC errors. laying out components.
Connections:
- net 3V3: now also R_NTC1.1, R_NTC2.1
Changed lines of the file:
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@@
 	)
 	(global_label "5V_DAC"
-		(shape input)
+		(shape output)
 		(at 158.75 157.48 0)
 		(fields_autoplaced yes)
@@
 	(global_label "3V3"
 		(shape input)
-		(at 183.93 67.12 180)
-		(fields_autoplaced yes)
-		(effects
-			(font
-				(size 1.27 1.27)
-			)
-			(justify right)
-		)
-		(property "Intersheetrefs" "${INTERSHEET_REFS}"
-			(at 183.93 67.12 0)
+		(at 184.15 67.31 180)
+		(fields_autoplaced yes)
+		(effects
+			(font
+				(size 1.27 1.27)
+			)
+			(justify right)
+		)
+		(property "Intersheetrefs" "${INTERSHEET_REFS}"
+			(at 184.15 67.31 0)
 			(hide yes)
 			(show_name no)
@@
 	(global_label "3V3"
 		(shape input)
-		(at 183.93 36.64 180)
-		(fields_autoplaced yes)
-		(effects
-			(font
-				(size 1.27 1.27)
-			)
-			(justify right)
-		)
-		(property "Intersheetrefs" "${INTERSHEET_REFS}"
-			(at 183.93 36.64 0)
+		(at 184.15 36.83 180)
+		(fields_autoplaced yes)
+		(effects
+			(font
+				(size 1.27 1.27)
+			)
+			(justify right)
+		)
+		(property "Intersheetrefs" "${INTERSHEET_REFS}"
+			(at 184.15 36.83 0)
 			(hide yes)
 			(show_name no)
@@
 		(property "Reference" "U29"
 			(at 140.97 151.13 0)
+			(hide yes)
 			(show_name no)
 			(do_not_autoplace no)
@@
 		(property "Value" "OPA2141AID"
 			(at 141.478 153.162 0)
+			(hide yes)
 			(show_name no)
 			(do_not_autoplace no)
@@
 		)
 		(property "Footprint" "Package_SO:SOIC-8_3.9x4.9mm_P1.27mm"
-			(at 139.7 165.1 0)
+			(at 140.462 178.054 0)
 			(hide yes)
 			(show_name no)
@@
 		(pin "4"
 		)
-		(pin "6"
-		)
-		(pin "8"
-		)
-		(pin "4"
-		)
-		(pin "5"
-		)
-		(pin "7"
-		)
 		(instances

Commit message: Added separate xfrmer for 6V.
Added inrush protection with NTC and increased capacitance to reduce ripple on 6V
Parts:
- renumbered J1 to J2, J2 to J3, R74 to R88, R75 to R89, R76 to R90, R77 to R91, R78 to R92, R79 to R93
Changed lines of the file:
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@@
 		(in_pos_files yes)
 		(dnp no)
-		(property "Reference" "R76"
+		(property "Reference" "R90"
 			(at 56.642 171.45 90)
 			(show_name no)
@@
 			(project "laser_driver_v3"
 				(path "/b2c3d4e5-f6a7-8901-bcde-f12345678901/e2f6689f-2746-4fd7-aa4a-0128f1e05d63"
-					(reference "R76")
+					(reference "R90")
 					(unit 1)
 				)
@@
 		(in_pos_files yes)
 		(dnp no)
-		(property "Reference" "J2"
+		(property "Reference" "J3"
 			(at 30.48 143.8031 0)
 			(show_name no)
@@
 			(project "laser_driver_v3"
 				(path "/b2c3d4e5-f6a7-8901-bcde-f12345678901/e2f6689f-2746-4fd7-aa4a-0128f1e05d63"
-					(reference "J2")
+					(reference "J3")
 					(unit 1)
 				)
@@
 		(in_pos_files yes)
 		(dnp no)
-		(property "Reference" "R79"
+		(property "Reference" "R93"
 			(at 115.57 75.692 90)
 			(show_name no)
@@
 			(project "laser_driver_v3"
 				(path "/b2c3d4e5-f6a7-8901-bcde-f12345678901/e2f6689f-2746-4fd7-aa4a-0128f1e05d63"
-					(reference "R79")
+					(reference "R93")
 					(unit 1)
 				)
@@
 		(in_pos_files yes)
 		(dnp no)
-		(property "Reference" "R75"
+		(property "Reference" "R89"
 			(at 39.37 71.882 90)
 			(show_name no)
@@
 			(project "laser_driver_v3"
 				(path "/b2c3d4e5-f6a7-8901-bcde-f12345678901/e2f6689f-2746-4fd7-aa4a-0128f1e05d63"
-					(reference "R75")
+					(reference "R89")
 					(unit 1)
 				)
@@
 		(in_pos_files yes)
 		(dnp no)
-		(property "Reference" "R77"
+		(property "Reference" "R91"
 			(at 57.912 132.08 90)
 			(show_name no)
@@
 			(project "laser_driver_v3"
 				(path "/b2c3d4e5-f6a7-8901-bcde-f12345678901/e2f6689f-2746-4fd7-aa4a-0128f1e05d63"
-					(reference "R77")
+					(reference "R91")
 					(unit 1)
 				)
@@
 		(in_pos_files yes)
 		(dnp no)
-		(property "Reference" "J1"
+		(property "Reference" "J2"
 			(at 29.21 183.1731 0)
 			(show_name no)
@@
 			(project "laser_driver_v3"
 				(path "/b2c3d4e5-f6a7-8901-bcde-f12345678901/e2f6689f-2746-4fd7-aa4a-0128f1e05d63"
-					(reference "J1")
+					(reference "J2")
 					(unit 1)
 				)
@@
 		(in_pos_files yes)
 		(dnp no)
-		(property "Reference" "R78"
+		(property "Reference" "R92"
 			(at 114.3 43.942 90)
 			(show_name no)
@@
 			(project "laser_driver_v3"
 				(path "/b2c3d4e5-f6a7-8901-bcde-f12345678901/e2f6689f-2746-4fd7-aa4a-0128f1e05d63"
-					(reference "R78")
+					(reference "R92")
 					(unit 1)
 				)
@@
 		(in_pos_files yes)
 		(dnp no)
-		(property "Reference" "R74"
+		(property "Reference" "R88"
 			(at 39.37 43.942 90)
 			(show_name no)
@@
 			(project "laser_driver_v3"
 				(path "/b2c3d4e5-f6a7-8901-bcde-f12345678901/e2f6689f-2746-4fd7-aa4a-0128f1e05d63"
-					(reference "R74")
-					(unit 1)
-				)
+					(reference "R88")
+					(unit 1)
+				)

Commit message: Changed xfrmers, paralled BJTs for cap multiplier
Changed the transformers to more appropriate voltages.
Made the BJTs for the cap multipliers in parallel to better handle the load.
Simulated the output ripple for the 6V.
Clarifying notes, removed LT1028 changed to OPA192 to match circuit as drawn.
Changed divider values for the TEC_zero value to be 1.2 V as designed.
Parts:
- renumbered R88 to R90, R89 to R91, R90 to R92, R91 to R93, R92 to R94, R93 to R95
Other:
- note added: "INA826 gains: Laser G=103.7 (Rg=487, Vmax=2.59V@100mA) TEC G=7.2 (Rg=8.06k, Vmax=3.0V@2.5A)"
- note removed: "INA826 gains: Laser G=106 (Rg=487, Vmax=3.0V@600mA) TEC G=7.2 (Rg=8.06k, Vmax=3.0V@2.5A)"
Changed lines of the file:
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@@
 		)
 	)
-	(text "INA826 gains: Laser G=106 (Rg=487, Vmax=3.0V@600mA)  TEC G=7.2 (Rg=8.06k, Vmax=3.0V@2.5A)"
+	(text "INA826 gains: Laser G=103.7 (Rg=487, Vmax=2.59V@100mA)  TEC G=7.2 (Rg=8.06k, Vmax=3.0V@2.5A)"
 		(exclude_from_sim no)
 		(at 14.478 17.272 0)
@@
 		(in_pos_files yes)
 		(dnp no)
-		(property "Reference" "R90"
+		(property "Reference" "R92"
 			(at 56.642 171.45 90)
 			(show_name no)
@@
 			(project "laser_driver_v3"
 				(path "/b2c3d4e5-f6a7-8901-bcde-f12345678901/e2f6689f-2746-4fd7-aa4a-0128f1e05d63"
-					(reference "R90")
+					(reference "R92")
 					(unit 1)
 				)
@@
 		(in_pos_files yes)
 		(dnp no)
-		(property "Reference" "R93"
+		(property "Reference" "R95"
 			(at 115.57 75.692 90)
 			(show_name no)
@@
 			(project "laser_driver_v3"
 				(path "/b2c3d4e5-f6a7-8901-bcde-f12345678901/e2f6689f-2746-4fd7-aa4a-0128f1e05d63"
-					(reference "R93")
+					(reference "R95")
 					(unit 1)
 				)
@@
 		(in_pos_files yes)
 		(dnp no)
-		(property "Reference" "R89"
+		(property "Reference" "R91"
 			(at 39.37 71.882 90)
 			(show_name no)
@@
 			(project "laser_driver_v3"
 				(path "/b2c3d4e5-f6a7-8901-bcde-f12345678901/e2f6689f-2746-4fd7-aa4a-0128f1e05d63"
-					(reference "R89")
+					(reference "R91")
 					(unit 1)
 				)
@@
 		(in_pos_files yes)
 		(dnp no)
-		(property "Reference" "R91"
+		(property "Reference" "R93"
 			(at 57.912 132.08 90)
 			(show_name no)
@@
 			(project "laser_driver_v3"
 				(path "/b2c3d4e5-f6a7-8901-bcde-f12345678901/e2f6689f-2746-4fd7-aa4a-0128f1e05d63"
-					(reference "R91")
+					(reference "R93")
 					(unit 1)
 				)
@@
 		(in_pos_files yes)
 		(dnp no)
-		(property "Reference" "R92"
+		(property "Reference" "R94"
 			(at 114.3 43.942 90)
 			(show_name no)
@@
 			(project "laser_driver_v3"
 				(path "/b2c3d4e5-f6a7-8901-bcde-f12345678901/e2f6689f-2746-4fd7-aa4a-0128f1e05d63"
-					(reference "R92")
+					(reference "R94")
 					(unit 1)
 				)
@@
 		(in_pos_files yes)
 		(dnp no)
-		(property "Reference" "R88"
+		(property "Reference" "R90"
 			(at 39.37 43.942 90)
 			(show_name no)
@@
 			(project "laser_driver_v3"
 				(path "/b2c3d4e5-f6a7-8901-bcde-f12345678901/e2f6689f-2746-4fd7-aa4a-0128f1e05d63"
-					(reference "R88")
+					(reference "R90")
 					(unit 1)
 				)

Commit message: Many changes.  Working through ERC.
Main changes are for the grounds.  I found the NETTIE function to tie the GND, DGND and AGND together at a specific point on the boud with a footprint even.
Changed transformers one more time to be consistent for both.
Updated footprints to be consistent and avoid power input/output errors with the ERC.
Changed lines of the file:
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@@
 	)
 	(junction
-		(at 201.93 50.8)
-		(diameter 0)
-		(color 0 0 0 0)
-	)
-	(junction
 		(at 260.35 130.81)
 		(diameter 0)
@@
 	)
 	(junction
-		(at 201.93 81.28)
-		(diameter 0)
-		(color 0 0 0 0)
-	)
-	(junction
 		(at 41.91 171.45)
 		(diameter 0)
@@
 	(wire
 		(pts
-			(xy 190.5 50.8) (xy 201.93 50.8)
+			(xy 190.5 50.8) (xy 229.87 50.8)
 		)
 		(stroke
@@
 	(wire
 		(pts
-			(xy 201.93 48.26) (xy 201.93 50.8)
-		)
-		(stroke
-			(width 0)
-			(type default)
-		)
-	)
-	(wire
-		(pts
 			(xy 241.3 132.08) (xy 247.65 132.08)
 		)
@@
 	(wire
 		(pts
-			(xy 201.93 78.74) (xy 204.47 78.74)
-		)
-		(stroke
-			(width 0)
-			(type default)
-		)
-	)
-	(wire
-		(pts
 			(xy 45.72 45.72) (xy 39.37 45.72)
 		)
@@
 	(wire
 		(pts
-			(xy 201.93 78.74) (xy 201.93 81.28)
-		)
-		(stroke
-			(width 0)
-			(type default)
-		)
-	)
-	(wire
-		(pts
 			(xy 226.06 35.56) (xy 226.06 48.26)
 		)
@@
 	(wire
 		(pts
-			(xy 201.93 81.28) (xy 229.87 81.28)
-		)
-		(stroke
-			(width 0)
-			(type default)
-		)
-	)
-	(wire
-		(pts
 			(xy 213.36 119.38) (xy 209.55 119.38)
 		)
@@
 	(wire
 		(pts
-			(xy 201.93 50.8) (xy 229.87 50.8)
-		)
-		(stroke
-			(width 0)
-			(type default)
-		)
-	)
-	(wire
-		(pts
 			(xy 95.25 182.88) (xy 101.6 182.88)
 		)
@@
 	(wire
 		(pts
-			(xy 190.5 81.28) (xy 201.93 81.28)
+			(xy 190.5 81.28) (xy 229.87 81.28)
 		)
 		(stroke
@@
 		)
 	)
-	(global_label "NTC1_MON"
-		(shape input)
-		(at 201.93 48.26 0)
-		(fields_autoplaced yes)
-		(effects
-			(font
-				(size 1.27 1.27)
-			)
-			(justify left)
-		)
-		(property "Intersheetrefs" "${INTERSHEET_REFS}"
-			(at 201.93 48.26 0)
-			(hide yes)
-			(show_name no)
-			(do_not_autoplace no)
-			(effects
-				(font
-					(size 1.27 1.27)
-				)
-				(justify left)
-			)
-		)
-	)
 	(global_label "LAS1_IMON"
 		(shape input)
@@
 	)
 	(global_label "NTC1_A"
-		(shape input)
+		(shape passive)
 		(at 184.15 50.8 180)
 		(fields_autoplaced yes)
@@
 		)
 		(property "Intersheetrefs" "${INTERSHEET_REFS}"
-			(at 184.15 50.8 0)
+			(at 175.4423 50.8 0)
 			(hide yes)
 			(show_name no)
@@
 		)
 	)
-	(global_label "NTC2_MON"
-		(shape input)
-		(at 204.47 78.74 0)
-		(fields_autoplaced yes)
-		(effects
-			(font
-				(size 1.27 1.27)
-			)
-			(justify left)
-		)
-		(property "Intersheetrefs" "${INTERSHEET_REFS}"
-			(at 204.47 78.74 0)
-			(hide yes)
-			(show_name no)
-			(do_not_autoplace no)
-			(effects
-				(font
-					(size 1.27 1.27)
-				)
-				(justify left)
-			)
-		)
-	)
 	(global_label "TEC2_SENSE_N"
 		(shape output)
@@
 	)
 	(global_label "NTC2_A"
-		(shape input)
+		(shape passive)
 		(at 184.15 81.28 180)
 		(fields_autoplaced yes)
@@
 		)
 		(property "Intersheetrefs" "${INTERSHEET_REFS}"
-			(at 184.15 81.28 0)
+			(at 175.4423 81.28 0)
 			(hide yes)
 			(show_name no)
@@
 	)
 	(symbol
+		(lib_name "OPA380_4")
 		(lib_id "Amplifier_Operational:OPA380")
 		(at 254 130.81 0)
@@
 	)
 	(symbol
+		(lib_name "OPA380_1")
 		(lib_id "Amplifier_Operational:OPA380")
 		(at 58.42 182.88 0)
@@
 	)
 	(symbol
+		(lib_name "OPA380_3")
 		(lib_id "Amplifier_Operational:OPA380")
 		(at 207.01 132.08 0)
@@
 	)
 	(symbol
+		(lib_name "OPA380_2")
 		(lib_id "Amplifier_Operational:OPA380")
 		(at 59.69 143.51 0)
@@
 	)
 	(symbol
+		(lib_name "OPA380_5")
 		(lib_id "Amplifier_Operational:OPA380")
 		(at 236.22 49.53 0)

Commit message: 6 V supply. Annotations. Teensy zero current.
Connections:
- net LAS1_SENSE_N: now also U25.1 (-); no longer U25.4 (+)
- net LAS1_SENSE_P: now also U25.4 (+); no longer U25.1 (-)
- net LAS2_SENSE_N: now also U26.1 (-); no longer U26.4 (+)
- net LAS2_SENSE_P: now also U26.4 (+); no longer U26.1 (-)
- net Laser_VZERO renamed GND
