File: Lasser_Driver_v5/AC_Board/AC_Board.kicad_pcb (KiCad board)
At the start: 2 copper layers, 62.4 x 42.7 mm, 9 parts, among them J1 Screw_Terminal_01x03, J2 Screw_Terminal_01x03, J3 Screw_Terminal_01x03

Commit message: Updates to AC board and pm22V prior to order
Parts:
- J1, J2, J3: footprint Connector_Phoenix_MSTB:PhoenixContact_MSTBA_2,5_3-G-5,08_1x03_P5.08mm_Horizontal -> TerminalBlock_Phoenix:TerminalBlock_Phoenix_MKDS-1,5-3-5.08_1x03_P5.08mm_Horizontal
