File: Lasser_Driver_v5/pm22V/pm22V.kicad_pcb (KiCad board)
At the start: 2 copper layers, 160 x 100 mm, 28 parts, among them J5 Screw_Terminal_01x03, J6 DIN41612_M_3x8+8_Power_Male, Q1 IRF540NPBF, Q2 IRF9540NPBF

Commit message: Updates to AC board and pm22V prior to order
Parts:
- J5: footprint Connector_Phoenix_MSTB:PhoenixContact_MSTBA_2,5_3-G-5,08_1x03_P5.08mm_Horizontal -> TerminalBlock_Phoenix:TerminalBlock_Phoenix_MKDS-1,5-3-5.08_1x03_P5.08mm_Horizontal
- moved C10 51.3 mm to (196.3, 123.5)
Routing:
- net /RAW22+: track 146.7 -> 164.2 mm

Commit message: Fixed PM22V bridge rectifier footprint.
Routing:
- net /RAW22-: track 101.8 -> 122.3 mm
- net -18Vac: track 31.7 -> 42.1 mm
Changed lines of the file:
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@@
 		(sheetname "/")
 		(sheetfile "pm22V.kicad_sch")
-		(units
-			(unit
-				(name "A")
-				(pins "4" "2" "3" "1")
-			)
-		)
 		(attr through_hole)
 		(duplicate_pad_numbers_are_jumpers no)
@@
 		)
 		(pad "3" thru_hole circle
-			(at 18 11.6)
+			(at 18 -6.4)
 			(size 2.8 2.8)
 			(drill 1.4)
@@
 		)
 		(pad "4" thru_hole circle
-			(at 18 -6.4)
+			(at 18 11.6)
 			(size 2.8 2.8)
 			(drill 1.4)
@@
 	)
 	(via
-		(at 201 89.5)
+		(at 199.44 85.34)
 		(size 0.8)
 		(drill 0.4)
@@
 	)
 	(via
-		(at 176.2 66.9)
+		(at 176.66 74.03)
 		(size 0.8)
 		(drill 0.4)
@@
 	)
 	(via
-		(at 196.1 83.7)
+		(at 206.32 85.47)
 		(size 0.8)
 		(drill 0.4)
@@
 	)
 	(segment
-		(start 206 74)
-		(end 193 74)
+		(start 194.35 79.95)
+		(end 194.35 90.65)
 		(width 1.5)
 		(layer "B.Cu")
@@
 	)
 	(segment
-		(start 193 74)
-		(end 187 80)
+		(start 194.35 90.65)
+		(end 187 98)
 		(width 1.5)
 		(layer "B.Cu")
@@
 	(segment
 		(start 209 65)
-		(end 209 71)
+		(end 209 65.3)
 		(width 1.5)
 		(layer "B.Cu")
@@
 	)
 	(segment
-		(start 209 71)
-		(end 206 74)
+		(start 209 65.3)
+		(end 194.35 79.95)
 		(width 1.5)
 		(layer "B.Cu")
@@
 	)
 	(segment
-		(start 187 98)
-		(end 181 104)
-		(width 2.5)
-		(layer "F.Cu")
-		(net "/RAW22-")
-	)
-	(segment
-		(start 181 104)
-		(end 168.92 104)
-		(width 2.5)
-		(layer "F.Cu")
-		(net "/RAW22-")
-	)
-	(segment
 		(start 128 72.9)
 		(end 128 62.28)
@@
 	)
 	(segment
+		(start 163.21 110.13)
+		(end 163 109.92)
+		(width 2.5)
+		(layer "B.Cu")
+		(net "/RAW22-")
+	)
+	(segment
 		(start 163 109.92)
 		(end 160.48 109.92)
@@
 	)
 	(segment
+		(start 164.61 109.92)
+		(end 187 87.53)
+		(width 2.5)
+		(layer "B.Cu")
+		(net "/RAW22-")
+	)
+	(segment
+		(start 187 87.53)
+		(end 187 80)
+		(width 2.5)
+		(layer "B.Cu")
+		(net "/RAW22-")
+	)
+	(segment
+		(start 163 109.92)
+		(end 164.61 109.92)
+		(width 2.5)
+		(layer "B.Cu")
+		(net "/RAW22-")
+	)
+	(segment
 		(start 151.6 118.8)
 		(end 151.6 126.2)
@@
 		(polygon
 			(pts
-				(xy 160.5 111) (xy 165.2 111.1) (xy 165.2 106.9) (xy 169.706237 104.772055) (xy 169.889584 102.480221)
-				(xy 160.5 104.8)
+				(xy 160.5 111) (xy 165.2 111.1) (xy 166.65 107.04) (xy 177.523255 105.677193) (xy 178.019273 103.632386)
+				(xy 160.94 104.36)
 			)
 		)
