File: Lasser_Driver_v5/pm1p8V_pm5V_5Vref_5Vlaser/pm1p8V_pm5V_5Vref_5Vlaser.kicad_sch (KiCad schematic)
At the start: 95 parts, among them J6 DIN41612_M_3x8+8_Power_Male, U1 MC7808CTG, U10 LT3042EMSE +14.3V, U13 MC7812CTG, U14 MC7808CTG, U15 LT3045EMSE 5V, U16 LT3045EMSE 5V, U17 MC7808CTG, U18 LM7905_TO220, U19 LT3045EMSE 5V, U2 LT3042EMSE +5.5V, U20 LT3094EMSE -5V, U21 OPA192IDBVR, U3 LTC6655BHMS8-5#PBF, U4 MC7812CTG, U5 MC7805CTG, U6 LT3045EMSE 3.3V, U7 LP5907MFX-1.8, U8 TPS7A3901DSCR, U9 LT3094EMSE -14.3V

Commit message: Continued work on power booards.
Parts:
- added C75: 1uF, Capacitor_SMD:C_0805_2012Metric_Pad1.18x1.45mm_HandSolder, symbol Device:C
- added HS1, HS2, HS3, HS4, HS5, HS6: Heatsink Boyd 531102B02500G, Heatsink:Heatsink_AAVID_Extruded_531102B02500G_34.9x12.7mm_H38.1mm, symbol Mechanical:Heatsink
- added R50: 49.9R, Resistor_SMD:R_0805_2012Metric_Pad1.20x1.40mm_HandSolder, symbol Device:R
- R10: value 54.9k 0.1% -> 60.4k 0.1%; DigiKey P/N P54.9KDATR-ND -> P60.4KDATR-ND; Manufacturer Part Number ERA-6AEB5492V -> ERA-6AEB6042V
- R11: value 1k -> 0R; DigiKey P/N 541-1.00KCTR-ND -> 311-0.0ARTR-ND; Manufacturer Vishay Dale -> YAGEO; Manufacturer Part Number CRCW08051K00FKEA -> RC0805JR-070RL
- R15: value 12.7k 0.1% -> 137k 0.1%; DigiKey P/N P12.7KDATR-ND -> 10-ERA-6AEB1373VTR-ND; Manufacturer Part Number ERA-6AEB1272V -> ERA-6AEB1373V
- R16: value 1k -> 10k 0.1%; DigiKey P/N 541-1.00KCTR-ND -> P10KDATR-ND; Manufacturer Vishay Dale -> Panasonic Industry; Manufacturer Part Number CRCW08051K00FKEA -> ERA-6AEB103V
- R41: value 49.9k 0.1% -> 24.9k 0.1%; DigiKey P/N P49.9KDATR-ND -> P24.9KDATR-ND; Manufacturer Part Number ERA-6AEB4992V -> ERA-6AEB2492V
- R44: value 16k -> 604; DigiKey P/N 311-16.0KCRTR-ND -> 311-604CRTR-ND; Manufacturer Part Number RC0805FR-0716KL -> RC0805FR-07604RL
- R48, R49: value 10k -> 10k 0.1%; DigiKey P/N 311-10.0KCRTR-ND -> P10KDATR-ND; Manufacturer YAGEO -> Panasonic Industry; Manufacturer Part Number RC0805FR-0710KL -> ERA-6AEB103V
- U18: value LM7905_TO220 -> MC7906CTG; DigiKey P/N MC7905CTGOS-ND -> MC7906CTGOS-ND; Manufacturer Part Number MC7905CTG -> MC7906CTG
Connections:
- net +5V: no longer R48.2
- net -5V: no longer R49.1
- net 5Vref: now also R48.2
- net GND: now also R49.1, C75.2; no longer C59.1, R16.2, R40.2, U15.1 (IN), U15.2 (IN), U15.3 (IN), U15.4 (EN/UV), U15.7 (PGFB), U16.1 (IN), U16.2 (IN), U16.3 (IN), U16.4 (EN/UV), U16.7 (PGFB)
- net VREF_MID: now also R50.2; no longer U21.1 (OUT), U21.2 (IN-)
- net at U8.8 (BUF): now also R16.2
- net at R48.1, R49.2, U21.3 (IN+): now also C75.1
- new net: C59.1, R40.2, U15.1 (IN), U15.2 (IN), U15.3 (IN), U15.4 (EN/UV), U15.7 (PGFB), U16.1 (IN), U16.2 (IN), U16.3 (IN), U16.4 (EN/UV), U16.7 (PGFB)
- new net: R50.1, U21.1 (OUT), U21.2 (IN-)
- no-connect marks 24 -> 23
Other:
- moved on the sheet: C25, C26, C27, C28, C29, C30, C31, C32, C33, C72, C73, C74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

Commit message: Power cards should be done now.
This should be the last power card.  Need to do one last review, but routing seems to be good.
Parts:
- R42, R43: value 20m PCB Trace -> 20m 1%; DigiKey P/N (none) -> P.02AQTR-ND; Manufacturer (none) -> Panasonic Industry; Manufacturer Part Number (none) -> ERJ-6BWFR020V; now fitted
Connections:
- removed net DGND: J6.P2, J6.P4, J6.a20
- no-connect marks 23 -> 32
