File: Lasser_Driver_v5/pm6V/pm6V.kicad_sch (KiCad schematic)
At the start: 62 parts, among them J4 Screw_Terminal_01x03, J6 DIN41612_M_3x8+8_Power_Male, Q10 Q_NPN MJL21194, Q3 IRF540NPBF, Q4 IRF9540NPBF, Q5 MMBT2907, Q6 MMBT2222, Q7 Q_PNP_MJL21193, Q8 Q_PNP_MJL21193, Q9 Q_NPN MJL21194, U11 LM4051AIM3-ADJ/NOPB, U12 LM4051AIM3-ADJ/NOPB

Commit message: pm6V v5 update
Parts:
- added HS2, HS3: Heatsink Boyd 531102B02500G, Heatsink:Heatsink_AAVID_Extruded_531102B02500G_34.9x12.7mm_H38.1mm, symbol Mechanical:Heatsink
Changed lines of the file:
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@@
+	)
+	(symbol
+		(lib_id "Mechanical:Heatsink")
+		(at 133.35 30.48 0)
+		(unit 1)
+		(body_style 1)
+		(exclude_from_sim no)
+		(in_bom yes)
+		(on_board yes)
+		(in_pos_files yes)
+		(dnp no)
+		(property "Reference" "HS2"
+			(at 135.89 25.4 0)
+			(show_name no)
+			(do_not_autoplace no)
+			(effects
+				(font
+					(size 1.27 1.27)
+				)
+			)
+		)
+		(property "Value" "Heatsink Boyd 531102B02500G"
+			(at 134.62 32.258 0)
+			(show_name no)
+			(do_not_autoplace no)
+			(effects
+				(font
+					(size 1.27 1.27)
+				)
+			)
+		)
+		(property "Footprint" "Heatsink:Heatsink_AAVID_Extruded_531102B02500G_34.9x12.7mm_H38.1mm"
+			(at 133.35 30.48 0)
+			(hide yes)
+			(show_name no)
+			(do_not_autoplace no)
+			(effects
+				(font
+					(size 1.27 1.27)
+				)
+			)
+		)
+		(property "Datasheet" ""
+			(at 133.35 30.48 0)
+			(hide yes)
+			(show_name no)
+			(do_not_autoplace no)
+			(effects
+				(font
+					(size 1.27 1.27)
+				)
+			)
+		)
+		(property "Description" "Heatsink TO-220 board-mount, DK HS352-ND"
+			(at 133.35 30.48 0)
+			(hide yes)
+			(show_name no)
+			(do_not_autoplace no)
+			(effects
+				(font
+					(size 1.27 1.27)
+				)
+			)
+		)
+		(instances
+			(project "pm6V"
+				(path "/e63e39d7-6ac0-4ffd-8aa3-1841a4541b55"
+					(reference "HS2")
+					(unit 1)
+				)
+			)
+		)
+	)
+	(symbol
+		(lib_id "Mechanical:Heatsink")
+		(at 133.35 60.96 0)
+		(unit 1)
+		(body_style 1)
+		(exclude_from_sim no)
+		(in_bom yes)
+		(on_board yes)
+		(in_pos_files yes)
+		(dnp no)
+		(property "Reference" "HS3"
+			(at 135.89 55.88 0)
+			(show_name no)
+			(do_not_autoplace no)
+			(effects
+				(font
+					(size 1.27 1.27)
+				)
+			)
+		)
+		(property "Value" "Heatsink Boyd 531102B02500G"
+			(at 134.62 62.738 0)
+			(show_name no)
+			(do_not_autoplace no)
+			(effects
+				(font
+					(size 1.27 1.27)
+				)
+			)
+		)
+		(property "Footprint" "Heatsink:Heatsink_AAVID_Extruded_531102B02500G_34.9x12.7mm_H38.1mm"
+			(at 133.35 60.96 0)
+			(hide yes)
+			(show_name no)
+			(do_not_autoplace no)
+			(effects
+				(font
+					(size 1.27 1.27)
+				)
+			)
+		)
+		(property "Datasheet" ""
+			(at 133.35 60.96 0)
+			(hide yes)
+			(show_name no)
+			(do_not_autoplace no)
+			(effects
+				(font
+					(size 1.27 1.27)
+				)
+			)
+		)
+		(property "Description" "Heatsink TO-220 board-mount, DK HS352-ND"
+			(at 133.35 60.96 0)
+			(hide yes)
+			(show_name no)
+			(do_not_autoplace no)
+			(effects
+				(font
+					(size 1.27 1.27)
+				)
+			)
+		)
+		(instances
+			(project "pm6V"
+				(path "/e63e39d7-6ac0-4ffd-8aa3-1841a4541b55"
+					(reference "HS3")
+					(unit 1)
+				)
+			)
+		)
 	)
 	(symbol

Commit message: pm6V PCB finished.  Started last power board.
Parts:
- C34, C35, C36, C37, C38, C39: footprint Capacitor_THT:C_Radial_D16.0mm_H25.0mm_P7.50mm -> Capacitor_THT:CP_Radial_D16.0mm_P7.50mm; DigiKey P/N (none) -> 493-1568-ND; Manufacturer (none) -> Nichicon; Manufacturer Part Number (none) -> UHE1E332MHD
- C40, C41, C48, C49, C50, C51: DigiKey P/N (none) -> 493-1557-ND; Manufacturer (none) -> Nichicon; Manufacturer Part Number (none) -> UHE1E102MPD
- C42, C43: DigiKey P/N (none) -> 1276-1039-2-ND; Manufacturer (none) -> Samsung; Manufacturer Part Number (none) -> CL21B474KBFNNNE
- C44, C45, C52, C53: DigiKey P/N (none) -> 1276-CL21B225KBYNNWETR-ND; Manufacturer (none) -> Samsung; Manufacturer Part Number (none) -> CL21B225KBYNNWE
- C46, C47: DigiKey P/N (none) -> 493-1346-ND; Manufacturer (none) -> Nichicon; Manufacturer Part Number (none) -> UVZ1H222MHD
- D10, D11, D_CP1, D_CP2: DigiKey P/N (none) -> 1N4148W-FDITR-ND; Manufacturer (none) -> Diodes Incorporated; Manufacturer Part Number (none) -> 1N4148W-7-F
- D7: value GBPC1510-E4/51 -> GBPC1510W-E4/51; DigiKey P/N (none) -> 2616-GBPC1510W-ND; Manufacturer (none) -> Surge Components; Manufacturer Part Number (none) -> GBPC1510W
- D8, D9: DigiKey P/N (none) -> 1N4742AFSTR-ND; Manufacturer (none) -> onsemi; Manufacturer Part Number (none) -> 1N4742ATR
- HS1: DigiKey P/N (none) -> 6223BG-ND; Manufacturer (none) -> Boyd; Manufacturer Part Number (none) -> 6223BG
- HS2, HS3: DigiKey P/N (none) -> HS352-ND; Manufacturer (none) -> Boyd; Manufacturer Part Number (none) -> 531102B02500G
- J4: DigiKey P/N (none) -> 277-1248-ND; Manufacturer Part Number (none) -> 1729131
- J6: DigiKey P/N (none) -> 2684-374144-E-ND; Manufacturer (none) -> TE Connectivity; Manufacturer Part Number (none) -> 374144-E
- Q10, Q9: footprint Heatsinks:TO-264-3_Vertical_HS657-25ABPE -> Heatsinks:TO-264-3_Vertical_HS657-10ABPE; DigiKey P/N (none) -> MJL21194GOS-ND; Manufacturer (none) -> onsemi; Manufacturer Part Number (none) -> MJL21194G
- Q3: value IRF540NPBF -> IRF540ZPBF; DigiKey P/N (none) -> IRF540ZPBF-ND; Manufacturer (none) -> Infineon; Manufacturer Part Number (none) -> IRF540ZPBF
- Q4: DigiKey P/N (none) -> IRF9540NPBF-ND; Manufacturer (none) -> Infineon; Manufacturer Part Number (none) -> IRF9540NPBF
- Q5: DigiKey P/N (none) -> MMBT2907A-TPMSTR-ND; Manufacturer (none) -> MCC; Manufacturer Part Number (none) -> MMBT2907A-TP
- Q6: DigiKey P/N (none) -> MMBT2222ALT1GOSTR-ND; Manufacturer (none) -> onsemi; Manufacturer Part Number (none) -> MMBT2222ALT1G
- Q7, Q8: footprint Heatsinks:TO-264-3_Vertical_HS657-25ABPE -> Heatsinks:TO-264-3_Vertical_HS657-10ABPE; DigiKey P/N (none) -> MJL21193GOS-ND; Manufacturer (none) -> onsemi; Manufacturer Part Number (none) -> MJL21193G
- R20, R21: DigiKey P/N (none) -> TUW15J15RE-ND; Manufacturer (none) -> Ohmite; Manufacturer Part Number (none) -> TUW15J15RE
- R22, R23: DigiKey P/N (none) -> 311-100KCRTR-ND; Manufacturer (none) -> YAGEO; Manufacturer Part Number (none) -> RC0805FR-07100KL
- R24, R31: DigiKey P/N (none) -> 311-15.0KCRTR-ND; Manufacturer (none) -> YAGEO; Manufacturer Part Number (none) -> RC0805FR-0715KL
- R25, R30: DigiKey P/N (none) -> P60.4KCTR-ND; Manufacturer (none) -> Panasonic; Manufacturer Part Number (none) -> ERJ-6ENF6042V
- R26, R27: DigiKey P/N (none) -> 311-1.00MCRTR-ND; Manufacturer (none) -> YAGEO; Manufacturer Part Number (none) -> RC0805FR-071ML
- R28, R29: DigiKey P/N (none) -> 311-1.50KCRTR-ND; Manufacturer (none) -> YAGEO; Manufacturer Part Number (none) -> RC0805FR-071K5L
- R34, R35, R36, R37: DigiKey P/N (none) -> WSLG-.10TR-ND; Manufacturer (none) -> Vishay Dale; Manufacturer Part Number (none) -> WSL2512R1000FEA
- R38, R39: DigiKey P/N (none) -> 541-1.00KCTR-ND; Manufacturer (none) -> Vishay Dale; Manufacturer Part Number (none) -> CRCW08051K00FKEA
- R40, R41, R42, R43: DigiKey P/N (none) -> 311-10.0CRTR-ND; Manufacturer (none) -> YAGEO; Manufacturer Part Number (none) -> RC0805FR-0710RL
- U11, U12: DigiKey P/N (none) -> LM4051AIM3-ADJ/NOPBTR-ND; Manufacturer (none) -> Texas Instruments; Manufacturer Part Number (none) -> LM4051AIM3-ADJ/NOPB
Connections:
- net DGND: now also C37.1, C38.1, C39.1, C41.1; no longer C37.2, C38.2, C39.2, C41.2
- net TEC_RAW-: now also C37.2, C38.2, C39.2, C41.2; no longer C37.1, C38.1, C39.1, C41.1
Other:
- moved on the sheet: C37, C38, C39, C41, HS2, HS3

Commit message: Continued work on power booards.
Parts:
- R24, R31: value 15k -> 60.4k; DigiKey P/N 311-15.0KCRTR-ND -> P60.4KCTR-ND; Manufacturer YAGEO -> Panasonic; Manufacturer Part Number RC0805FR-0715KL -> ERJ-6ENF6042V
- R25, R30: value 60.4k -> 15k; DigiKey P/N P60.4KCTR-ND -> 311-15.0KCRTR-ND; Manufacturer Panasonic -> YAGEO; Manufacturer Part Number ERJ-6ENF6042V -> RC0805FR-0715KL
Changed lines of the file:
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@@
 			)
 		)
-		(property "Value" "60.4k"
+		(property "Value" "15k"
 			(at 158.242 163.322 0)
 			(show_name no)
@@
 			)
 		)
-		(property "Manufacturer Part Number" "ERJ-6ENF6042V"
+		(property "Manufacturer Part Number" "RC0805FR-0715KL"
 			(at 163.322 165.1 0)
 			(hide yes)
@@
 			)
 		)
-		(property "Manufacturer" "Panasonic"
+		(property "Manufacturer" "YAGEO"
 			(at 163.322 165.1 0)
 			(hide yes)
@@
 			)
 		)
-		(property "DigiKey P/N" "P60.4KCTR-ND"
+		(property "DigiKey P/N" "311-15.0KCRTR-ND"
 			(at 163.322 165.1 0)
 			(hide yes)
@@
 			)
 		)
-		(property "Value" "60.4k"
+		(property "Value" "15k"
 			(at 144.018 124.968 0)
 			(show_name no)
@@
 			)
 		)
-		(property "Manufacturer Part Number" "ERJ-6ENF6042V"
+		(property "Manufacturer Part Number" "RC0805FR-0715KL"
 			(at 138.938 123.19 0)
 			(hide yes)
@@
 			)
 		)
-		(property "Manufacturer" "Panasonic"
+		(property "Manufacturer" "YAGEO"
 			(at 138.938 123.19 0)
 			(hide yes)
@@
 			)
 		)
-		(property "DigiKey P/N" "P60.4KCTR-ND"
+		(property "DigiKey P/N" "311-15.0KCRTR-ND"
 			(at 138.938 123.19 0)
 			(hide yes)
@@
 			)
 		)
-		(property "Value" "15k"
+		(property "Value" "60.4k"
 			(at 159.766 171.958 0)
 			(show_name no)
@@
 			)
 		)
-		(property "Manufacturer Part Number" "RC0805FR-0715KL"
+		(property "Manufacturer Part Number" "ERJ-6ENF6042V"
 			(at 163.322 173.99 0)
 			(hide yes)
@@
 			)
 		)
-		(property "Manufacturer" "YAGEO"
+		(property "Manufacturer" "Panasonic"
 			(at 163.322 173.99 0)
 			(hide yes)
@@
 			)
 		)
-		(property "DigiKey P/N" "311-15.0KCRTR-ND"
+		(property "DigiKey P/N" "P60.4KCTR-ND"
 			(at 163.322 173.99 0)
 			(hide yes)
@@
 			)
 		)
-		(property "Value" "15k"
+		(property "Value" "60.4k"
 			(at 142.494 116.332 0)
 			(show_name no)
@@
 			)
 		)
-		(property "Manufacturer Part Number" "RC0805FR-0715KL"
+		(property "Manufacturer Part Number" "ERJ-6ENF6042V"
 			(at 138.938 114.3 0)
 			(hide yes)
@@
 			)
 		)
-		(property "Manufacturer" "YAGEO"
+		(property "Manufacturer" "Panasonic"
 			(at 138.938 114.3 0)
 			(hide yes)
@@
 			)
 		)
-		(property "DigiKey P/N" "311-15.0KCRTR-ND"
+		(property "DigiKey P/N" "P60.4KCTR-ND"
 			(at 138.938 114.3 0)
 			(hide yes)

Commit message: Figured out remaining cards.
Created backplane pcb.  Should be ready to go to fab just need BOM.  Layout matches standard for hole spacing.
Updated Teensy code to match pinout and updated schematics.
Changed DGND to TECGND for clarity.
Connections:
- net DGND renamed PGND_TEC
Changed lines of the file:
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@@
 		)
 	)
-	(global_label "DGND"
+	(global_label "PGND_TEC"
 		(shape passive)
 		(at 106.68 176.53 0)
@@
 		)
 	)
-	(global_label "DGND"
+	(global_label "PGND_TEC"
 		(shape passive)
 		(at 38.1 27.94 0)
@@
 		)
 	)
-	(global_label "DGND"
+	(global_label "PGND_TEC"
 		(shape passive)
 		(at 267.97 46.99 0)
@@
 		)
 	)
-	(global_label "DGND"
+	(global_label "PGND_TEC"
 		(shape passive)
 		(at 267.97 41.91 0)
@@
 		)
 	)
-	(global_label "DGND"
+	(global_label "PGND_TEC"
 		(shape passive)
 		(at 266.7 127 0)
@@
 		)
 	)
-	(global_label "DGND"
+	(global_label "PGND_TEC"
 		(shape passive)
 		(at 193.04 38.1 0)
@@
 		)
 	)
-	(global_label "DGND"
+	(global_label "PGND_TEC"
 		(shape passive)
 		(at 127 81.28 0)
