File: Lasser_Driver_v5/CH_Card/CH_Card.kicad_sch (KiCad schematic)
At the start: 143 parts, among them J1 DIN41612_M_universal, Q13 IRL540N, Q14 IRF9540N, Q17 IRL540N, Q18 IRF9540N, Q19 DMN3404L, U101 AD5696R, U102 ADS1115, U103 PCA9538, U104 ADG419BRM, U105 ADG419BRM, U17 OPA192IDBVR, U19 OPA192IDBVR, U21 OPA551U, U22 OPA192IDBVR, U24 OPA192IDBVR, U26 ADG419BRM, U28 INA828, U32 INA828

Commit message: Progress on the laser card.
Update photodiode monitoring.
Parts:
- added H1, H2: MountingHole, MountingHole:MountingHole_2.7mm, symbol Mechanical:MountingHole
- added HS1: 657-10ABPE (Q13), symbol Mechanical:Heatsink
- added HS2: 657-10ABPE (Q14), symbol Mechanical:Heatsink
- added HS3: 657-10ABPE (Q17), symbol Mechanical:Heatsink
- added HS4: 657-10ABPE (Q18), symbol Mechanical:Heatsink
- Q13, Q14, Q17, Q18: footprint Package_TO_SOT_THT:TO-220-3_Vertical -> Heatsinks:TO-220-3_Vertical_HS657-10ABPE
- R68, R76: value 47R prot -> 10mR link (was 47R - TEC path); footprint Resistor_SMD:R_0805_2012Metric_Pad1.20x1.40mm_HandSolder -> Resistor_SMD:R_2512_6332Metric
- R73, R74: value 47R prot -> 0R link (was 47R - laser path)
- R_bias1: value 100k PD bias -> 20k 0.1% PD bias; footprint Resistor_SMD:R_0805_2012Metric_Pad1.20x1.40mm_HandSolder -> Resistor_SMD:R_0805_2012Metric
Connections:
- net unconnected-(J_BTF1-NC-Pad3) is gone; now on net GND: J_BTF1.3 (NC)
- net unconnected-(J_BTF1-NC-Pad4) is gone; now on net MPD_K: J_BTF1.4 (NC)
Other:
- note added: "TEC H-BRIDGE HEATSINKS: HS1-HS4 = Wakefield 657-10ABPE on Q13/Q14/Q17/Q18 (combined footprint Heatsinks:TO-220-3_Vertical_HS657-10ABPE carries the copper - HS symbols are BOM-only). Isolate every tab: Boyd 4880G kit + #4-40 screw/washers/nut. Worst case ~10W/FET at 2.5A TEC cooling. Fins vertical; keep away from NTC divider + precision scalers."
- moved on the sheet: C132, C133, C134, C135, C136, C137, C139, C142, C143, C144, C145, C146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

Commit message: Progress on laying out the laser PCB
Parts:
- added R78: 100k, Resistor_SMD:R_0805_2012Metric_Pad1.20x1.40mm_HandSolder, symbol Device:R
- J_BTF1: value DFB1550LP #1 Socket -> Butterfly harness header - Wurth WR-PHD 2x7 (mates LDM-BUTTERFLY); footprint Connector_PinSocket_2.54mm:PinSocket_2x07_P2.54mm_Vertical -> Connector_PinHeader_2.54mm:PinHeader_2x07_P2.54mm_Vertical
Connections:
- net GND: now also R78.1
- net N_C70_~_Pad1: now also R78.2
- net TEC_BTF_N: no longer R62.2
Other:
- moved on the sheet: R44

Commit message: Working on the CH pcb layout and routing.
Parts:
- removed R62: DNP Rtrim (shunt scale), Resistor_SMD:R_0805_2012Metric_Pad1.20x1.40mm_HandSolder, symbol Device:R
Changed lines of the file:
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@@
 	)
 	(junction
-		(at 382.27 212.09)
-		(diameter 0)
-		(color 0 0 0 0)
-	)
-	(junction
 		(at 82.55 210.82)
 		(diameter 0)
@@
 	(wire
 		(pts
-			(xy 382.27 209.55) (xy 382.27 212.09)
-		)
-		(stroke
-			(width 0)
-			(type default)
-		)
-	)
-	(wire
-		(pts
 			(xy 143.51 207.01) (xy 143.51 208.28)
 		)
@@
 	(wire
 		(pts
-			(xy 382.27 212.09) (xy 387.35 212.09)
-		)
-		(stroke
-			(width 0)
-			(type default)
-		)
-	)
-	(wire
-		(pts
 			(xy 388.62 128.27) (xy 388.62 130.81)
 		)
@@
 	(wire
 		(pts
-			(xy 382.27 212.09) (xy 382.27 224.79)
+			(xy 382.27 209.55) (xy 382.27 224.79)
 		)
 		(stroke
@@
 		(pin "7"
 		)
+		(pin "8"
+		)
+		(pin "5"
+		)
+		(pin "1"
+		)
 		(instances
 			(project "CH_Card"
@@
 	)
 	(symbol
-		(lib_id "Device:R")
-		(at 387.35 215.9 0)
-		(unit 1)
-		(body_style 1)
-		(exclude_from_sim no)
-		(in_bom yes)
-		(on_board yes)
-		(in_pos_files yes)
-		(dnp yes)
-		(property "Reference" "R62"
-			(at 387.858 215.392 0)
-			(show_name no)
-			(do_not_autoplace no)
-			(effects
-				(font
-					(size 1.27 1.27)
-				)
-			)
-		)
-		(property "Value" "DNP Rtrim (shunt scale)"
-			(at 387.604 217.17 0)
-			(show_name no)
-			(do_not_autoplace no)
-			(effects
-				(font
-					(size 1.27 1.27)
-				)
-			)
-		)
-		(property "Footprint" "Resistor_SMD:R_0805_2012Metric_Pad1.20x1.40mm_HandSolder"
-			(at 387.35 215.9 0)
-			(hide yes)
-			(show_name no)
-			(do_not_autoplace no)
-			(effects
-				(font
-					(size 1.27 1.27)
-				)
-			)
-		)
-		(property "Datasheet" ""
-			(at 387.35 215.9 0)
-			(hide yes)
-			(show_name no)
-			(do_not_autoplace no)
-			(effects
-				(font
-					(size 1.27 1.27)
-				)
-			)
-		)
-		(property "Description" ""
-			(at 387.35 215.9 0)
-			(show_name no)
-			(do_not_autoplace no)
-			(effects
-				(font
-					(size 1.27 1.27)
-				)
-			)
-		)
-		(pin "1"
-		)
-		(pin "2"
-		)
-		(instances
-			(project "CH_Card"
-				(path "/2abe37a0-24c0-47ee-a2b1-3dcf608486c0"
-					(reference "R62")
-					(unit 1)
-				)
-			)
-		)
-	)
-	(symbol
 		(lib_id "Device:C")
 		(at 54.61 182.88 0)
@@
 		)
 		(property "Footprint" "Package_SO:SOIC-8_3.9x4.9mm_P1.27mm"
-			(at 542.29 53.34 0)
+			(at 545.338 36.576 0)
 			(hide yes)
 			(show_name no)
@@
 		(pin "3"
 		)
+		(pin "1"
+		)
+		(pin "8"
+		)
+		(pin "5"
+		)
 		(instances
