File: Lasser_Driver_v5/Backplane/Backplane_Slots.kicad_pcb (KiCad board)
At the start: 2 copper layers, 390.4 x 128.6 mm, 24 parts, among them J1 294711-E, J2 294711-E, J3 294711-E, J4 294711-E, J5 294711-E, J6 294711-E, J7 294711-E, J8 294711-E

Commit message: Changed CH card to 6 layer. Added single pt grnd.
CH card is now layed out cleanly with 6 layers.
Added a single point connection with surge protection to the backplane.
Parts:
- added C1: 100n, Capacitor_SMD:C_0805_2012Metric_Pad1.18x1.45mm_HandSolder, F.Cu at (405.2, 108.8)
- added D3: SMAJ5.0CA, Diode_SMD:D_SMA-SMB_Universal_Handsoldering, F.Cu at (408.6, 108.8)
- added R1: 0, Resistor_SMD:R_0805_2012Metric_Pad1.20x1.40mm_HandSolder, F.Cu at (402.9, 108.7)
Connections:
- J1 pad a20: GA2 -> unconnected-(J1-Pada20)
- J1 pad c18: GA0 -> unconnected-(J1-Padc18)
- J1 pad c19: GA1 -> unconnected-(J1-Padc19)
- J2 pad a20: GA2 -> unconnected-(J2-Pada20)
- J2 pad c18: GA0 -> unconnected-(J2-Padc18)
- J2 pad c19: GA1 -> unconnected-(J2-Padc19)
- J3 pad a20: GA2 -> unconnected-(J3-Pada20)
- J3 pad c18: GA0 -> unconnected-(J3-Padc18)
- J3 pad c19: GA1 -> unconnected-(J3-Padc19)
- J4 pad a20: GA2 -> unconnected-(J4-Pada20)
- J4 pad c18: GA0 -> unconnected-(J4-Padc18)
- J4 pad c19: GA1 -> unconnected-(J4-Padc19)
- J5 pad a20: GA2 -> unconnected-(J5-Pada20)
- J5 pad c18: GA0 -> unconnected-(J5-Padc18)
- J5 pad c19: GA1 -> unconnected-(J5-Padc19)
- J6 pad a20: GA2 -> unconnected-(J6-Pada20)
- J6 pad c18: GA0 -> unconnected-(J6-Padc18)
- J6 pad c19: GA1 -> unconnected-(J6-Padc19)
- J7 pad a20: GA2 -> unconnected-(J7-Pada20)
- J7 pad c18: GA0 -> unconnected-(J7-Padc18)
- J7 pad c19: GA1 -> unconnected-(J7-Padc19)
- J8 pad a20: GA2 -> unconnected-(J8-Pada20)
- J8 pad c18: GA0 -> unconnected-(J8-Padc18)
- J8 pad c19: GA1 -> unconnected-(J8-Padc19)
Routing:
- net +6V_TEC: track 661.6 -> 712.4 mm
- net PGND_TEC: track 1325.3 -> 1375.9 mm
- net GND: track 1621.9 -> 1636.1 mm
- net -6V_TEC: track 642.6 -> 645.9 mm
- net MOD2_DRV: track 580.7 -> 582.2 mm
- net +15V: track 374.5 -> 373.5 mm
- net +18V: track 570.8 -> 570.5 mm, vias 22 -> 21
- net -18V: vias 28 -> 27
- added copper zone on B.Cu, net GND
- added copper zone on F.Cu, net GND
- added copper zone on B.Cu, net PGND_TEC
- added copper zone on F.Cu, net PGND_TEC
