File: Lasser_Driver_v5/DIG_Card/DIG_Card.kicad_sch (KiCad schematic)
At the start: 173 parts, among them J2 10MHz Ref SMA, J301 DIN41612_M_universal, J302 LO1/LO2 out SMA, U301 OPA192IDBVR MOD1 buffer, U302 OPA192IDBVR MOD2 buffer, U303 74LVC1G125 CLK10M bus buffer, U34 AD9833xRM, U35 AD9833xRM (ref), U38 AD9833xRM (ref), U39 AD9833xRM, U40 LMV7219M5, U41 SN74LVC1G3157DBVR, U42 CDCE913PWG4, U44 CR2013-MI2120, Y1 ASE-10.000MHZ-LC-T

Commit message: working on the digital pcb layout.  Mostly done.
Parts:
- removed JP301: GA0 addr jumper, Connector_PinHeader_2.54mm:PinHeader_1x02_P2.54mm_Vertical, symbol DIGCard_New:JP_ADDR
- removed JP302: GA1 addr jumper, Connector_PinHeader_2.54mm:PinHeader_1x02_P2.54mm_Vertical, symbol DIGCard_New:JP_ADDR
- removed JP303: GA2 addr jumper, Connector_PinHeader_2.54mm:PinHeader_1x02_P2.54mm_Vertical, symbol DIGCard_New:JP_ADDR
- removed R308: 10k GA0 pullup, Resistor_SMD:R_0805_2012Metric, symbol Device:R
- removed R309: 10k GA1 pullup, Resistor_SMD:R_0805_2012Metric, symbol Device:R
- removed R310: 10k GA2 pullup, Resistor_SMD:R_0805_2012Metric, symbol Device:R
- added C312: 100nF Y1 3V3_OSC, Capacitor_SMD:C_0805_2012Metric, symbol Device:C
- added C313: 1uF Y1 3V3_OSC, Capacitor_SMD:C_0805_2012Metric, symbol Device:C
- added C314: 100nF U40 3V3, Capacitor_SMD:C_0805_2012Metric, symbol Device:C
- added C315: 100nF U41 3V3, Capacitor_SMD:C_0805_2012Metric, symbol Device:C
- added C316: 100nF U42 1V8, Capacitor_SMD:C_0805_2012Metric, symbol Device:C
- added C317: 100nF U42 3V3, Capacitor_SMD:C_0805_2012Metric, symbol Device:C
- added C318: 10uF U42 3V3, Capacitor_SMD:C_0805_2012Metric, symbol Device:C
- added C319: 1uF U42 1V8_CLK, Capacitor_SMD:C_0805_2012Metric, symbol Device:C
- added C92: 0.1uF, Capacitor_SMD:C_0805_2012Metric_Pad1.18x1.45mm_HandSolder, symbol Device:C
- added FB301: 600R@100MHz FB Y1, Inductor_SMD:L_0805_2012Metric, symbol Device:FerriteBead_Small
- added FB302: 600R@100MHz FB U42core, Inductor_SMD:L_0805_2012Metric, symbol Device:FerriteBead_Small
Connections:
- net 1V8: no longer U42.3 (VDD)
- net 3V3: now also C314.1, C315.1, C317.1, C318.1, C92.2, FB301.1; no longer Y1.1 (TRI-STATE(STBY)), Y1.4 (VDD)
- net GND: now also C312.2, C313.2, C314.2, C315.2, C316.2, C317.2, C318.2, C319.2, C92.1
- net VM_N_R58_Pad1: now also D304.1 (K), VM_R58.1, VM_R98.1, VM_U23.13
- net GA0: no longer names the net of A1.D14 (A0)
- net GA0_BP: no longer names the net of J301.c18
- net GA1: no longer names the net of A1.D15 (A1)
- net GA1_BP: no longer names the net of J301.c19
- net GA2: no longer names the net of A1.D16 (A2)
- net GA2_BP: no longer names the net of J301.a20
- new net: C312.1, C313.1, FB301.2, Y1.1 (TRI-STATE(STBY))
- new net: C316.1, C319.1, FB302.1, U42.3 (VDD)
- new net 1V8_CLK: FB302.2
- new net 3V3_OSC: Y1.4 (VDD)
- no-connect marks 27 -> 33
Other:
- note removed: "I don't think this card needs jumpers for the address."
- note removed: "why pullup here, aren't there pullup resistors on other cards?"
- moved on the sheet: R111, U42

Commit message: Working on digital card.
Put a bunch of vias, but didn't set the net to GND.  Need to make them all GND.
Parts:
- removed unit 2 of J2
- removed unit 2 of J302
- added J302B1: Conn_Coaxial, Connector_Coaxial:SMA_BAT_Wireless_BWSMA-KWE-Z001, symbol Connector:Conn_Coaxial
- added R114: 100, Resistor_SMD:R_0805_2012Metric_Pad1.20x1.40mm_HandSolder, symbol Device:R
- J2: symbol Connector:Conn_Coaxial_x2_Isolated -> Connector:Conn_Coaxial
- J302: value LO1/LO2 out SMA -> LO1 out SMA; symbol Connector:Conn_Coaxial_x2_Isolated -> Connector:Conn_Coaxial
Connections:
- net 1V8: now also FB302.2
- net 1V8_CLK: now also C316.1, C319.1, FB302.1, U42.3 (VDD); no longer FB302.2
- net 3V3: now also R114.2; no longer U44.8 (LED)
- net 3V3_OSC: now also C313.1
- net GND: now also J302B1.2 (Ext)
- net LO2_OUT: now also J302B1.1 (In)
- net at C312.1, FB301.2, Y1.1 (TRI-STATE(STBY)): no longer C313.1
- new net: R114.1, U44.8 (LED)
- no-connect marks 33 -> 31
Other:
- moved on the sheet: C313

Commit message: Many updates to the digital PCB
Made LO outs 50 ohm
Added 100 ohm resistor to display LED
Added 33 0hm resistors to clocks 2 and 3 to prevent ringing
Fixed traces, no connects, etc.
Added ground vias.
Parts:
- added R316: 33R MCLK2 series, Resistor_SMD:R_0805_2012Metric, symbol Device:R
- added R317: 33R MCLK3 series, Resistor_SMD:R_0805_2012Metric, symbol Device:R
- VM_U22: value MCP6002-xMC -> MCP6002-xSN; symbol Amplifier_Operational:MCP6002-xMC -> Amplifier_Operational:MCP6002-xSN
Connections:
- net GND: no longer VM_U22.9 (V-)
- net MCLK2: now also R316.2; no longer U42.9 (Y2)
- net MCLK3: now also R317.2; no longer U42.8 (Y3)
- new net MCLK2_S: R316.1, U42.9 (Y2)
- new net MCLK3_S: R317.1, U42.8 (Y3)
Changed lines of the file:
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@@
 		)
 	)
-	(label "MCLK3"
+	(label "MCLK3_S"
 		(at 384.81 335.28 0)
 		(effects
@@
 		)
 	)
-	(label "VM_N_U28A__"
-		(at 708.66 1120.14 0)
-		(effects
-			(font
-				(size 1.27 1.27)
-			)
-			(justify left)
-		)
-	)
 	(label "N_C90_Pad2"
 		(at 297.18 259.08 180)
@@
 		)
 	)
-	(label "MCLK2"
+	(label "MCLK2_S"
 		(at 384.81 331.47 0)
 		(effects
@@
 		)
 	)
-	(label "VM_N_D21_K"
-		(at 758.19 416.56 270)
-		(effects
-			(font
-				(size 1.27 1.27)
-			)
-			(justify right)
-		)
-	)
 	(label "VM_N_R102_Pad1"
 		(at 654.05 417.83 0)
@@
 	)
 	(symbol
-		(lib_id "Amplifier_Operational:MCP6002-xMC")
+		(lib_id "Amplifier_Operational:MCP6002-xSN")
 		(at 684.53 60.96 0)
 		(unit 2)
@@
 			)
 		)
-		(property "Value" "MCP6002-xMC"
+		(property "Value" "MCP6002-xSN"
 			(at 691.134 64.77 0)
 			(show_name no)
@@
 		(pin "4"
 		)
-		(pin "9"
-		)
 		(pin "7"
 		)
@@
 	)
 	(symbol
-		(lib_id "Amplifier_Operational:MCP6002-xMC")
+		(lib_id "Amplifier_Operational:MCP6002-xSN")
 		(at 378.46 55.88 0)
 		(unit 3)
@@
 			)
 		)
-		(property "Value" "MCP6002-xMC"
+		(property "Value" "MCP6002-xSN"
 			(at 380.746 56.642 0)
 			(show_name no)
@@
 		(pin "2"
 		)
-		(pin "9"
-		)
 		(instances
 			(project "DIG_Card"
@@
 	)
 	(symbol
-		(lib_id "Amplifier_Operational:MCP6002-xMC")
+		(lib_id "Amplifier_Operational:MCP6002-xSN")
 		(at 684.53 48.26 0)
 		(unit 1)
@@
 			)
 		)
-		(property "Value" "MCP6002-xMC"
+		(property "Value" "MCP6002-xSN"
 			(at 691.642 52.07 0)
 			(show_name no)
@@
 		(pin "6"
 		)
-		(pin "9"
-		)
 		(pin "3"
 		)
@@
 	)
 	(embedded_fonts no)
+	(label "MCLK2_S"
+		(at 394.97 320.0 180)
+		(effects
+			(font
+				(size 1.27 1.27)
+			)
+			(justify right)
+		)
+	)
+	(label "MCLK2"
+		(at 402.59 320.0 0)
+		(effects
+			(font
+				(size 1.27 1.27)
+			)
+			(justify left)
+		)
+	)
+	(label "MCLK3_S"
+		(at 394.97 340.0 180)
+		(effects
+			(font
+				(size 1.27 1.27)
+			)
+			(justify right)
+		)
+	)
+	(label "MCLK3"
+		(at 402.59 340.0 0)
+		(effects
+			(font
+				(size 1.27 1.27)
+			)
+			(justify left)
+		)
+	)
+	(symbol
+		(lib_id "Device:R")
+		(at 398.78 320.0 90)
+		(unit 1)
+		(body_style 1)
+		(exclude_from_sim no)
+		(in_bom yes)
+		(on_board yes)
+		(in_pos_files yes)
+		(dnp no)
+		(property "Reference" "R316"
+			(at 398.78 320.0 90)
+			(show_name no)
+			(do_not_autoplace no)
+			(effects
+				(font
+					(size 1.27 1.27)
+				)
+			)
+		)
+		(property "Value" "33R MCLK2 series"
+			(at 406.4 322.286 90)
+			(show_name no)
+			(do_not_autoplace no)
+			(effects
+				(font
+					(size 1.27 1.27)
+				)
+			)
+		)
+		(property "Footprint" "Resistor_SMD:R_0805_2012Metric"
+			(at 398.78 320.0 0)
+			(hide yes)
+			(show_name no)
+			(do_not_autoplace no)
+			(effects
+				(font
+					(size 1.27 1.27)
+				)
+			)
+		)
+		(property "Datasheet" ""
+			(at 398.78 320.0 0)
+			(hide yes)
+			(show_name no)
+			(do_not_autoplace no)
+			(effects
+				(font
+					(size 1.27 1.27)
+				)
+			)
+		)
+		(property "Description" ""
+			(at 398.78 320.0 0)
+			(show_name no)
+			(do_not_autoplace no)
+			(effects
+				(font
+					(size 1.27 1.27)
+				)
+			)
+		)
+		(pin "1"
+		)
+		(pin "2"
+		)
+		(instances
+			(project "DIG_Card"
+				(path "/ba312f5e-b1e5-475d-8676-33718a7f94d0"
+					(reference "R316")
+					(unit 1)
+				)
+			)
+		)
+	)
+	(symbol
+		(lib_id "Device:R")
+		(at 398.78 340.0 90)
+		(unit 1)
+		(body_style 1)
+		(exclude_from_sim no)
+		(in_bom yes)
+		(on_board yes)
+		(in_pos_files yes)
+		(dnp no)
+		(property "Reference" "R317"
+			(at 398.78 340.0 90)
+			(show_name no)
+			(do_not_autoplace no)
+			(effects
+				(font
+					(size 1.27 1.27)
+				)
+			)
+		)
+		(property "Value" "33R MCLK3 series"
+			(at 406.4 342.286 90)
+			(show_name no)
+			(do_not_autoplace no)
+			(effects
+				(font
+					(size 1.27 1.27)
+				)
+			)
+		)
+		(property "Footprint" "Resistor_SMD:R_0805_2012Metric"
+			(at 398.78 340.0 0)
+			(hide yes)
+			(show_name no)
+			(do_not_autoplace no)
+			(effects
+				(font
+					(size 1.27 1.27)
+				)
+			)
+		)
+		(property "Datasheet" ""
+			(at 398.78 340.0 0)
+			(hide yes)
+			(show_name no)
+			(do_not_autoplace no)
+			(effects
+				(font
+					(size 1.27 1.27)
+				)
+			)
+		)
+		(property "Description" ""
+			(at 398.78 340.0 0)
+			(show_name no)
+			(do_not_autoplace no)
+			(effects
+				(font
+					(size 1.27 1.27)
+				)
+			)
+		)
+		(pin "1"
+		)
+		(pin "2"
+		)
+		(instances
+			(project "DIG_Card"
+				(path "/ba312f5e-b1e5-475d-8676-33718a7f94d0"
+					(reference "R317")
+					(unit 1)
+				)
+			)
+		)
+	)
 )

Commit message: Digital PCB improvements
Added more decoupling caps and bulk caps.  Layout for these done.
Added test point pads to the schematic.  Need to put these into the layout to make probing easy and clean.
Parts:
- added C320: 10nF U34 COMP, Capacitor_SMD:C_0805_2012Metric, symbol Device:C
- added C321: 10nF U39 COMP, Capacitor_SMD:C_0805_2012Metric, symbol Device:C
- added C322: 10uF +5V bulk, Capacitor_SMD:C_0805_2012Metric, symbol Device:C
- added C323: 10uF 3V3 bulk, Capacitor_SMD:C_0805_2012Metric, symbol Device:C
- added C324: 100nF 1V8 entry, Capacitor_SMD:C_0805_2012Metric, symbol Device:C
- added C325: 10uF 1V8 entry, Capacitor_SMD:C_0805_2012Metric, symbol Device:C
- added TP301: N_U41_B1, TestPoint:TestPoint_Pad_D1.0mm, symbol Connector:TestPoint
- added TP302: N_U41_A, TestPoint:TestPoint_Pad_D1.0mm, symbol Connector:TestPoint
- added TP303: CLK10M_BUF, TestPoint:TestPoint_Pad_D1.0mm, symbol Connector:TestPoint
- added TP304: MCLK1, TestPoint:TestPoint_Pad_D1.0mm, symbol Connector:TestPoint
- added TP305: MCLK2, TestPoint:TestPoint_Pad_D1.0mm, symbol Connector:TestPoint
- added TP306: 3V3_OSC, TestPoint:TestPoint_Pad_D1.0mm, symbol Connector:TestPoint
- added TP307: 1V8_CLK, TestPoint:TestPoint_Pad_D1.0mm, symbol Connector:TestPoint
- added TP308: 3V3, TestPoint:TestPoint_Pad_D1.0mm, symbol Connector:TestPoint
- added TP309: +5V, TestPoint:TestPoint_Pad_D1.0mm, symbol Connector:TestPoint
- added TP310: 1V8, TestPoint:TestPoint_Pad_D1.0mm, symbol Connector:TestPoint
- added TP311: 5Vref, TestPoint:TestPoint_Pad_D1.0mm, symbol Connector:TestPoint
- added TP312: VREF_MID, TestPoint:TestPoint_Pad_D1.0mm, symbol Connector:TestPoint
- added TP313: VHI_Buf, TestPoint:TestPoint_Pad_D1.0mm, symbol Connector:TestPoint
- added TP314: VLO_Buf, TestPoint:TestPoint_Pad_D1.0mm, symbol Connector:TestPoint
- added TP315, TP316, TP317, TP318, TP319, TP320: GND, TestPoint:TestPoint_THTPad_D1.5mm_Drill0.7mm, symbol Connector:TestPoint
Connections:
- net +5V: now also C322.1, TP309.1
- net 1V8: now also C324.1, C325.1, TP310.1
- net 1V8_CLK: now also TP307.1
- net 3V3: now also C323.1, TP308.1
- net 3V3_OSC: now also C312.1, FB301.2, Y1.1 (TRI-STATE(STBY)), TP306.1
- net 5Vref: now also TP311.1
- net CLK10M_BUF: now also TP303.1
- net GND: now also C320.2, C321.2, C322.2, C323.2, C324.2, C325.2, TP315.1, TP316.1, TP317.1, TP318.1, TP319.1, TP320.1
- net MCLK1: now also TP304.1
- net MCLK2: now also TP305.1
- net N_U41_A: now also TP302.1
- net N_U41_B1: now also TP301.1
- net VHI_Buf: now also TP313.1
- net VLO_Buf: now also TP314.1
- net VREF_MID: now also TP312.1
- net N_U34_COMP: now reaches U34.1 (COMP)
- net N_U34_COMP: now also C320.1
- net N_U39_COMP: now reaches U39.1 (COMP)
- net N_U39_COMP: now also C321.1
- no-connect marks 31 -> 29

Commit message: Finished the Digital card.
Layout and routing done.  Updated documentation.
Parts:
- TP313: value VHI_Buf -> VHI
- TP314: value VLO_Buf -> VLO
Changed lines of the file:
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@@
 			)
 		)
-		(property "Value" "VHI_Buf"
+		(property "Value" "VHI"
 			(at 398.78000000000003 409.92 0)
 			(show_name no)
@@
 			)
 		)
-		(property "Value" "VLO_Buf"
+		(property "Value" "VLO"
 			(at 414.02000000000004 409.92 0)
 			(show_name no)
