File: Lasser_Driver_v5/AFE_Card/AFE_Card.kicad_sch (KiCad schematic)
At the start: 144 parts, among them J1 DIN41612_M_universal, J202 PD1 pigtail, J203 PD2 pigtail, J204 LO4 ref SMA, J205 LO5 ref SMA, U1 LT3042EMSE +12V, U201 ADS1115, U202 OPA192IDBVR ERR1 buffer, U203 OPA192IDBVR ERR2 buffer, U204 OPA820 LOx3, U205 OPA820 LOx3, U206 AD5696R, U30 OPA859IDSGR, U31 OPA859IDSGR, U45 AD835 demod, U46 AD835 demod

Commit message: AFE card work.
Changed out TIA's and worked on routing.  No errors now.
Parts:
- removed C239: 100nF VREF1 filt, Capacitor_SMD:C_0805_2012Metric_Pad1.18x1.45mm_HandSolder, symbol Device:C
- removed C240: 100nF VREF2 filt, Capacitor_SMD:C_0805_2012Metric_Pad1.18x1.45mm_HandSolder, symbol Device:C
- removed C244: 10uF VREF_TIA bulk, Capacitor_SMD:C_0805_2012Metric_Pad1.18x1.45mm_HandSolder, symbol Device:C
- removed C245: 100nF VREF_TIA, Capacitor_SMD:C_0805_2012Metric_Pad1.18x1.45mm_HandSolder, symbol Device:C
- removed C246: 100nF VREF_TIA_ADC, Capacitor_SMD:C_0805_2012Metric_Pad1.18x1.45mm_HandSolder, symbol Device:C
- removed J202: PD1 pigtail, TerminalBlock_Phoenix:TerminalBlock_Phoenix_MKDS-1,5-3-5.08_1x03_P5.08mm_Horizontal, symbol Connector:Screw_Terminal_01x03
- removed J203: PD2 pigtail, TerminalBlock_Phoenix:TerminalBlock_Phoenix_MKDS-1,5-3-5.08_1x03_P5.08mm_Horizontal, symbol Connector:Screw_Terminal_01x03
- removed R130: 100R VREF1 filt, Resistor_SMD:R_0805_2012Metric_Pad1.20x1.40mm_HandSolder, symbol Device:R
- removed R131: 100R VREF2 filt, Resistor_SMD:R_0805_2012Metric_Pad1.20x1.40mm_HandSolder, symbol Device:R
- removed R132: 49.9k VREF_TIA top, Resistor_SMD:R_0805_2012Metric_Pad1.20x1.40mm_HandSolder, symbol Device:R
- removed R133: 100k VREF_TIA bot, Resistor_SMD:R_0805_2012Metric_Pad1.20x1.40mm_HandSolder, symbol Device:R
- removed R136: 10k VREF_TIA_ADC top, Resistor_SMD:R_0805_2012Metric_Pad1.20x1.40mm_HandSolder, symbol Device:R
- removed R137: 10k VREF_TIA_ADC bot, Resistor_SMD:R_0805_2012Metric_Pad1.20x1.40mm_HandSolder, symbol Device:R
- removed U30, U31: OPA859IDSGR, Package_SON:WSON-8-1EP_2x2mm_P0.5mm_EP0.9x1.6mm, symbol Amplifier_Operational:OPA859xDSG
- added C255: 100nF U30 -5V, Capacitor_SMD:C_0805_2012Metric_Pad1.18x1.45mm_HandSolder, symbol Device:C
- added C256: 100nF U31 -5V, Capacitor_SMD:C_0805_2012Metric_Pad1.18x1.45mm_HandSolder, symbol Device:C
- added PD1, PD2: FGA01FC, Optical:PD_TO46_FGA01FC_3pin, symbol Optical:PD_FGA01FC
- added U30, U31: OPA814DBVR, OPA814DBVR:OPA814DBVR, symbol OPA814DBVR:OPA814DBVR
- R118, R119: value 10k -> 6.65k
- TP412: value VREF_TIA -> 5Vref
- TP413: value VREF_TIA_1 -> PD1_LVL
- TP414: value VREF_TIA_2 -> PD2_LVL
Connections:
- net VREF_TIA is gone; now on net 5Vref: TP412.1
- net VREF_TIA_1 is gone; now on net PD1_LVL: TP413.1
- net VREF_TIA_2 is gone; now on net PD2_LVL: TP414.1
- net VREF_TIA_ADC is gone; now on net VREF_MID: U201.5 (AIN1), U201.7 (AIN3)
- net +5V: now also U30.5 (VS+), U31.5 (VS+)
- net -5V: now also C255.1, C256.1, U30.2 (VS-), U31.2 (VS-)
- net 5Vref: now also R134.2, R135.2
- net GND: now also U1.11 (Pad), C255.2, C256.2, PD1.2 (CASE), PD2.2 (CASE), U30.3 (IN+), U31.3 (IN+); no longer R134.2, R135.2
- net PD1_BIAS_K: now also PD1.1 (K)
- net PD1_IN: now also PD1.3 (A), U30.4 (IN-)
- net PD2_BIAS_K: now also PD2.1 (K)
- net PD2_IN: now also PD2.3 (A), U31.4 (IN-)
- net TIA1_OUT: now also U30.1 (OUT)
- net TIA2_OUT: now also U31.1 (OUT)
- net +6V_TEC: no longer names the net of J1.P1
- net -6V_TEC: no longer names the net of J1.P3
- net PGND_TEC: no longer names the net of J1.P2
- net PGND_TEC: no longer J1.P4
- no-connect marks 0 -> 4
Other:
- note added: "FGA01FC photodiodes (PD1/PD2) mount ON the front panel; only their three leads reach the board (Optical:PD_TO46_FGA01FC_3pin, 3 holes on a 2.5mm circle). Pin 1=K, 2=CASE, 3=A. Supplied with the optics - not on the BOM. The ANODE must sit millimetres from the TIA input: it is the compensated summing node (Cf 1pF), so place U30/U31 directly behind their diodes."
- note removed: "FGA01FC photodiodes are OFF-BOARD (fiber-coupled, front panel) - pigtails land on J202/J203 (sig/bias-K/shield)."

Commit message: Working on analog board.
Change photodiodes to the correct model and connector.  Made an adapter to allow the photodiode to be edge connect.  Made the footprint for the edge connect photodiode.  Updated estimates from capacitance and dark current specifications from photodiode.  Updates to manual and firmware correspond to all changes.
Moved libary of custom footprints to lib folder for easy finding.
Parts:
- PD1, PD2: footprint Optical:PD_TO46_FGA01FC_3pin -> Optical:PD_FGA01FC_EdgeBracket
Changed lines of the file:
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@@
 			)
 		)
-		(property "Footprint" "Optical:PD_TO46_FGA01FC_3pin"
+		(property "Footprint" "Optical:PD_FGA01FC_EdgeBracket"
 			(at 323.85 30.48 0)
 			(hide yes)
@@
 			)
 		)
-		(property "Footprint" "Optical:PD_TO46_FGA01FC_3pin"
+		(property "Footprint" "Optical:PD_FGA01FC_EdgeBracket"
 			(at 325.12 109.22 0)
 			(hide yes)

Commit message: updates to AFE, CH, DIG and pm1p8_pm5V_5Vlaser
schematics and pcbs updated.  They seem to be ready, but will take one more look with fresh eyes before ordering.
Parts:
- added C257: 10uF LT3042 IN bulk, Capacitor_SMD:C_0805_2012Metric_Pad1.18x1.45mm_HandSolder, symbol Device:C
- added C258: 100nF LT3042 IN, Capacitor_SMD:C_0805_2012Metric_Pad1.18x1.45mm_HandSolder, symbol Device:C
- J204: value LO4 ref SMA -> LO1 ref SMA
- J205: value LO5 ref SMA -> LO2 ref SMA
Connections:
- net +15V: now also C257.1, C258.1
- net GND: now also C257.2, C258.2
