File: Lasser_Driver_v6/CH_Card/CH_Card.kicad_sch (KiCad schematic)
At the start: 149 parts, among them J1 DIN41612_M_universal, Q13 IRL540N, Q14 IRF9540N, Q17 IRL540N, Q18 IRF9540N, Q19 DMN3404L, U101 AD5696R, U102 ADS1115, U103 PCA9538, U104 ADG419BRM, U105 ADG419BRM, U17 OPA192IDBVR, U19 OPA192IDBVR, U21 OPA551U, U22 OPA192IDBVR, U24 OPA192IDBVR, U26 ADG419BRM, U28 INA828, U32 INA828

Commit message: Main updates to CH card v6
Parts:
- added C167, C169, C173: 100nF +15V dec, Capacitor_SMD:C_0805_2012Metric_Pad1.18x1.45mm_HandSolder, symbol Device:C
- added C168, C170, C174: 100nF -15V dec, Capacitor_SMD:C_0805_2012Metric_Pad1.18x1.45mm_HandSolder, symbol Device:C
- added C171: 100nF loop comp, Capacitor_SMD:C_0805_2012Metric_Pad1.18x1.45mm_HandSolder, symbol Device:C
- added C172: 100nF -5V dec, Capacitor_SMD:C_0805_2012Metric_Pad1.18x1.45mm_HandSolder, symbol Device:C
- added D23: BAT46W flag clamp, Diode_SMD:D_SOD-123, symbol Device:D
- added R130: 10k inv in, Resistor_SMD:R_0805_2012Metric_Pad1.20x1.40mm_HandSolder, symbol Device:R
- added R131: 10k inv fb, Resistor_SMD:R_0805_2012Metric_Pad1.20x1.40mm_HandSolder, symbol Device:R
- added R132: 10R buf iso, Resistor_SMD:R_0805_2012Metric_Pad1.20x1.40mm_HandSolder, symbol Device:R
- added R133: 10k IMON fb, Resistor_SMD:R_0805_2012Metric_Pad1.20x1.40mm_HandSolder, symbol Device:R
- added R134: 15M pedestal cancel, Resistor_SMD:R_0805_2012Metric_Pad1.20x1.40mm_HandSolder, symbol Device:R
- added TP501: TEC_VZERO, TestPoint:TestPoint_Pad_D1.0mm, symbol Connector:TestPoint
- added TP502: N_U19_OUT, TestPoint:TestPoint_Pad_D1.0mm, symbol Connector:TestPoint
- added TP503: N_U19_INM, TestPoint:TestPoint_Pad_D1.0mm, symbol Connector:TestPoint
- added TP504: N_U106_OUT, TestPoint:TestPoint_Pad_D1.0mm, symbol Connector:TestPoint
- added TP505: N_U21__, TestPoint:TestPoint_Pad_D1.0mm, symbol Connector:TestPoint
- added TP506: N_U107_OUT, TestPoint:TestPoint_Pad_D1.0mm, symbol Connector:TestPoint
- added TP507: N_Q13_S, TestPoint:TestPoint_Pad_D1.0mm, symbol Connector:TestPoint
- added TP508: N_Q17_S, TestPoint:TestPoint_Pad_D1.0mm, symbol Connector:TestPoint
- added TP509: TEC_BTF_P, TestPoint:TestPoint_Pad_D1.0mm, symbol Connector:TestPoint
- added TP510: TEC_BTF_N, TestPoint:TestPoint_Pad_D1.0mm, symbol Connector:TestPoint
- added TP511: TEC_IMON, TestPoint:TestPoint_Pad_D1.0mm, symbol Connector:TestPoint
- added TP512: VOUT_LAS, TestPoint:TestPoint_Pad_D1.0mm, symbol Connector:TestPoint
- added TP513: N_U22_INP, TestPoint:TestPoint_Pad_D1.0mm, symbol Connector:TestPoint
- added TP514: N_Q19_S, TestPoint:TestPoint_Pad_D1.0mm, symbol Connector:TestPoint
- added TP515: LAS_IMON, TestPoint:TestPoint_Pad_D1.0mm, symbol Connector:TestPoint
- added TP516: N_U24_OUT, TestPoint:TestPoint_Pad_D1.0mm, symbol Connector:TestPoint
- added TP517: BTF_LASER, TestPoint:TestPoint_Pad_D1.0mm, symbol Connector:TestPoint
- added TP518: MPD_MON, TestPoint:TestPoint_Pad_D1.0mm, symbol Connector:TestPoint
- added TP519: NTC_A, TestPoint:TestPoint_Pad_D1.0mm, symbol Connector:TestPoint
- added TP520: TEC_EN, TestPoint:TestPoint_Pad_D1.0mm, symbol Connector:TestPoint
- added TP521: N_U21_Flag, TestPoint:TestPoint_Pad_D1.0mm, symbol Connector:TestPoint
- added TP522: LOCK_EN, TestPoint:TestPoint_Pad_D1.0mm, symbol Connector:TestPoint
- added TP523: VREF_MID, TestPoint:TestPoint_Pad_D1.0mm, symbol Connector:TestPoint
- added TP524: 5Vref, TestPoint:TestPoint_Pad_D1.0mm, symbol Connector:TestPoint
- added TP525: +5V_LASER, TestPoint:TestPoint_Pad_D1.0mm, symbol Connector:TestPoint
- added TP526: VZERO_SET, TestPoint:TestPoint_Pad_D1.0mm, symbol Connector:TestPoint
- added TP527, TP528, TP529, TP530: GND, TestPoint:TestPoint_THTPad_D1.5mm_Drill0.7mm, symbol Connector:TestPoint
- added U106: OPA192IDBVR, Package_TO_SOT_SMD:SOT-23-5, symbol LT1028_2
- added U107: OPA551U, Package_SO:SOIC-8_3.9x4.9mm_P1.27mm, symbol Amplifier_Operational:OPA551U
- added U108: ADG419BRM, Package_SO:MSOP-8_3x3mm_P0.65mm, symbol Analog_Switch:ADG419BRM
- R117: value 4.99k VZERO trim (v3 R40) -> 2.00k VZERO trim (v3 R40)
- R49: value 10k -> 33k flag pulldown
- R56, R57, R58, R59: value 47R -> 470R gate
- R67: value 1k 0.1% scaler_bot -> 909R 0.1% scaler_bot
- R96: value Rsum 10k -> Rsum 7.5M
Connections:
- net +15V: now also C167.1, C169.1, C173.1, U106.5 (V+), U107.7 (V+), U108.4 (V+)
- net +5V: now also U108.5 (VL)
- net +5V_LASER: now also TP525.1
- net -15V: now also C168.1, C170.1, C174.1, U106.2 (V-), U107.1 (V-), U107.4 (V-), U107.5 (V-), U108.7 (V-)
- net -5V: now also C172.1, R134.2
- net -6V_TEC: now also Q14.2 (D), Q18.2 (D); no longer Q14.3 (S), Q18.3 (S)
- net 3V3: now also D23.1 (K); no longer R49.1
- net 5Vref: now also TP524.1
- net BTF_LASER: now also TP517.1
- net FAULT_n: now also U102.2 (ALERT)
- net GND: now also R49.1, R67.1, C167.2, C168.2, C169.2, C170.2, C172.2, C173.2, C174.2, TP527.1, TP528.1, TP529.1, TP530.1, U106.3 (IN+), U108.3 (GND)
- net LAS_IMON: now also TP515.1
- net LOCK_EN: now also TP522.1
- net MPD_MON: now also TP518.1
- net NTC_A: now also TP519.1
- net N_Q13_S: now also Q14.3 (S), TP507.1; no longer Q14.2 (D)
- net N_Q17_S: now also Q18.3 (S), U32.4 (+), TP508.1; no longer Q18.2 (D), U32.1 (-)
- net N_Q19_S: now also TP514.1
- net N_U19_INP: now also C171.2, R133.2, U108.1
- net N_U19_OUT: now also C171.1, R130.1, TP502.1
- net N_U21_Flag: now also D23.2 (A), TP521.1, U107.8 (Flag)
- net N_U21__: now also TP505.1; no longer R57.1, R58.1
- net N_U22_INP: now also R96.2, R134.1, TP513.1
- net N_U24_OUT: now also TP516.1
- net TEC_BTF_N: now also TP510.1; no longer U19.4 (IN-)
- net TEC_BTF_P: now also U32.1 (-), TP509.1; no longer U32.4 (+)
- net TEC_IMON: now also R133.1, TP511.1
- net TEC_VZERO: now also TP501.1, U108.2
- net VOUT_LAS: now also TP512.1
- net VREF_MID: now also TP523.1
- net VZERO_SET: now also TP526.1
- removed net DITH_SUM: R67.1, R96.2
- net N_IO3 renamed TEC_EN
- net TEC_EN: now also TP520.1, U108.6
- new net: R132.2, U107.3 (+)
- new net N_U106_INM: R130.2, R131.1, U106.4 (IN-)
- new net N_U106_OUT: R131.2, R132.1, TP504.1, U106.1 (OUT)
- new net N_U107_OUT: R57.1, R58.1, TP506.1, U107.2 (-), U107.6
- new net N_U19_INM: TP503.1, U19.4 (IN-)
Other:
- note added: "Gate resistors are 470R, NOT 47R. On loop saturation each buffer drives its TWO gates toward +/-15 V into the D16/D17/D20/D21 forward clamps at +/-6.7 V: 47R -> (15-6.7)/(47/2) = 353 mA from a 200 mA OPA551 (current limit, then thermal shutdown) and 0.7 V x 353 mA = 247 mW in a 500 mW MMSZ4702. 470R -> 35 mA and 25 mW. Gate pole 70 ns -> 0.7 us, still ~2000x above the ~115 Hz TEC loop crossover, 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"
- note added: "Laser setpoint rev D: R67 909R is the scaler BOTTOM (to GND), not the servo tap. DAC 0-5V -> 22.62 mV at R81 0.25R -> 90.5 mA full scale (20 mW = 85.5 mA = 94.5% FS). PDH servo injects through R96 7.5M = 0.483 mA/V; an OPA192 railed to +14.8 V adds only +5.9 mA, so DAC full scale + a railed integrator = 96.4 mA, 3.6% under the DFB1550LP 100 mA absolute max. R134 15M to -5V cancels U24's 2.500 V V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"
- note added: "OPA551 Flag is a CURRENT SOURCE (<50 nA normal, 80/120/160 uA min/typ/max in thermal shutdown), NOT open-collector - so R49 is a PULL-DOWN, not a pull-up. normal 2 x 50 nA x 33k = 3.3 mV (< VIL 0.99 V); shutdown 80 uA x 33k = 2.64 V (> VIH 2.31 V). D23 BAT46W clamps the node to ~3.6 V so 160 uA (or both amps at once) cannot overdrive the PCA9538 input past its VDD+0.5 = 3.8 V abs max. U21 and U10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"
- note added: "TEC bridge rev D: leg 1 (Q13/Q14) driven by U106 inverter + U107 buffer; leg 2 (Q17/Q18) stays on U21, so the two legs swing in antiphase. Q14/Q18 mirrored: P-ch SOURCE on the bridge node, DRAIN on -6V_TEC. U19 closes on TEC_IMON (R133/C171 integrator, fc 159 Hz), not TEC_BTF_N. U32 inputs swapped so cooling reads ABOVE 1.20 V, per firmware config.h."
- note added: "TEC power-up safe state: U108 forces the setpoint node to TEC_VZERO = 0 A. A unipolar DAC needs a NONZERO code for zero current, so no U101 reset state can mean 'TEC off' - RSTSEL=GND boots the TEC to -1.34 A of heating, and RSTSEL=VLOGIC would fix that only by putting 45 mA of uncommanded current through the LASER. TEC_EN = PCA9538 IO3 with R121 10k to GND: the expander powers up with its IOs as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"
- note added: "TEST POINTS TP501-TP530 (this card previously had none). Signal pads TestPoint_Pad_D1.0mm; the four GND are THT so a scope ground spring clips on. DELIBERATELY EXCLUDED, do not 'add for completeness': the U24 PI summing node (N_U24_INP, C76 1n - a pad's stray C shifts the integrator) and the two MPD TIA inverting inputs (N_U_TIA1_IN_ / N_U_TIA2_IN_, where stray C detunes C_f1/C_f2). SDA/SCL/ERRn_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"

Commit message: updates to AFE, CH, DIG and pm1p8_pm5V_5Vlaser
schematics and pcbs updated.  They seem to be ready, but will take one more look with fresh eyes before ordering.
Connections:
- net N_U19_INM: now also C171.2, R133.2
- net N_U19_INP: no longer C171.2, R133.2
Changed lines of the file:
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@@
 	)
 	(junction
-		(at 241.3 184.15)
-		(diameter 0)
-		(color 0 0 0 0)
-	)
-	(junction
 		(at 271.78 275.59)
 		(diameter 0)
@@
 	)
 	(junction
-		(at 241.3 207.01)
-		(diameter 0)
-		(color 0 0 0 0)
-	)
-	(junction
 		(at 309.88 218.44)
 		(diameter 0)
@@
 	(wire
 		(pts
-			(xy 241.3 184.15) (xy 248.92 184.15)
-		)
-		(stroke
-			(width 0)
-			(type default)
-		)
-	)
-	(wire
-		(pts
 			(xy 673.1 137.16) (xy 670.56 137.16)
 		)
@@
 	(wire
 		(pts
-			(xy 237.49 184.15) (xy 241.3 184.15)
+			(xy 237.49 184.15) (xy 248.92 184.15)
 		)
 		(stroke
@@
 	(wire
 		(pts
-			(xy 241.3 184.15) (xy 241.3 207.01)
-		)
-		(stroke
-			(width 0)
-			(type default)
-		)
-	)
-	(wire
-		(pts
 			(xy 293.37 290.83) (xy 271.78 290.83)
 		)
@@
 		)
 	)
+	(label "N_U19_INM"
+		(at 241.3 209.55 0)
+		(effects
+			(font
+				(size 1.27 1.27)
+			)
+			(justify left bottom)
+		)
+	)
 	(label "TEC_EN"
 		(at 240.03 160.02 270)
@@
 		(dnp no)
 		(property "Reference" "C118"
-			(at 53.594 117.348 0)
+			(at 49.784 115.316 0)
 			(show_name no)
 			(do_not_autoplace no)
@@
 		)
 		(property "Value" "100nF decouple expander"
-			(at 63.754 121.92 0)
+			(at 53.848 119.38 90)
 			(show_name no)
 			(do_not_autoplace no)
