File: Lasser_Driver_v6/DIG_Card/DIG_Card.kicad_pcb (KiCad board)
At the start: 6 copper layers, 160 x 100 mm, 208 parts, among them J2 10MHz Ref SMA, J301 DIN41612_M_universal, J302 LO1 out SMA, J302B1 Conn_Coaxial, U301 OPA192IDBVR MOD1 buffer, U302 OPA192IDBVR MOD2 buffer, U303 74LVC1G125 CLK10M bus buffer, U34 AD9833xRM, U35 AD9833xRM (ref), U38 AD9833xRM (ref), U39 AD9833xRM, U40 LMV7219M5, U41 SN74LVC1G3157DBVR, U42 CDCE913PWG4, U44 CR2013-MI2120, Y1 ASE-10.000MHZ-LC-T

Commit message: Main updates to CH card v6
Changed lines of the file:
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@@
 		)
 		(property "Value" "1V8_CLK"
-			(at 0.05 -3.85 90)
+			(at 0.4 -3.85 90)
 			(layer "F.SilkS")
 			(effects
@@
 		)
 		(property "Value" "N_U41_A"
-			(at -0.05 -3.9 90)
+			(at 0.05 -3.35 90)
 			(layer "F.SilkS")
 			(effects

Commit message: updates to AFE, CH, DIG and pm1p8_pm5V_5Vlaser
schematics and pcbs updated.  They seem to be ready, but will take one more look with fresh eyes before ordering.
Parts:
- added R318: 33R MCLK1 series, Resistor_SMD:R_0805_2012Metric, B.Cu at (192.0, 73.0)
- J302B1: value Conn_Coaxial -> LO2 out SMA
- moved R114 0.43 mm to (146.7, 134.2)
- turned D24 to 0 degrees
Connections:
- D24 pad 1: /N_D24_A -> /N_D24_K_Pad1
- D24 pad 2: /N_D24_K_Pad1 -> unconnected-(D24-A-Pad2)
- D24 pad 3: unconnected-(D24-K-Pad3) -> /N_D24_A
- U42 pad 11: /MCLK1 -> /MCLK1_S
Routing:
- net /MCLK1_S: track 0.00 -> 2.75 mm, vias 0 -> 1
- net Net-(U44-LED): track 2.33 -> 3.18 mm
- net 3V3: track 530.7 -> 529.9 mm
- net /MCLK1: track 16.0 -> 16.2 mm, vias 0 -> 1
- net GND: vias 501 -> 505
