File: Lasser_Driver_v6/DIG_Card/DIG_Card.kicad_sch (KiCad schematic)
At the start: 208 parts, among them J2 10MHz Ref SMA, J301 DIN41612_M_universal, J302 LO1 out SMA, J302B1 Conn_Coaxial, U301 OPA192IDBVR MOD1 buffer, U302 OPA192IDBVR MOD2 buffer, U303 74LVC1G125 CLK10M bus buffer, U34 AD9833xRM, U35 AD9833xRM (ref), U38 AD9833xRM (ref), U39 AD9833xRM, U40 LMV7219M5, U41 SN74LVC1G3157DBVR, U42 CDCE913PWG4, U44 CR2013-MI2120, Y1 ASE-10.000MHZ-LC-T

Commit message: updates to AFE, CH, DIG and pm1p8_pm5V_5Vlaser
schematics and pcbs updated.  They seem to be ready, but will take one more look with fresh eyes before ordering.
Parts:
- added R318: 33R MCLK1 series, Resistor_SMD:R_0805_2012Metric, symbol Device:R
- J302B1: value Conn_Coaxial -> LO2 out SMA
Connections:
- net MCLK1: now also R318.2; no longer U42.11 (Y1)
- net N_D24_A: now also D24.3 (K); no longer D24.1 (K)
- net N_D24_K_Pad1: now also D24.1 (K); no longer D24.2 (A)
- new net MCLK1_S: R318.1, U42.11 (Y1)
Other:
- moved on the sheet: D24
