File: Laser_Driver_v7/AC_Board/AC_Board.kicad_sch (KiCad schematic)
At the start: 11 parts, among them J1 Screw_Terminal_01x03, J2 Screw_Terminal_01x03, J3 Screw_Terminal_01x03, T1 Triad VPT36-1390, T2 Triad VPT18-8800

Commit message: Working towards a full set of pcbs in v7
Parts:
- removed R1: 1k, Resistor_SMD:R_0805_2012Metric_Pad1.20x1.40mm_HandSolder, symbol Device:R
- TH1: footprint Resistor_THT:R_Axial_DIN0411_L9.9mm_D3.6mm_P7.62mm_Vertical -> Thermistor:Thermistor_Disc_D22.0mm_W5.0mm_P7.80mm_Ametherm_SL22
Connections:
- net at J3.2 (Pin_2): no longer J2.2 (Pin_2)
- no-connect marks 0 -> 2
