File: Laser_Driver_v7/AFE_Card/AFE_Card.kicad_sch (KiCad schematic)
At the start: 137 parts, among them J1 DIN41612_03x32_C_Split, J204 LO1 ref SMA, J205 LO2 ref SMA, U1 LT3042EMSE +12V, U201 ADS1115, U202 OPA192IDBVR ERR1 buffer, U203 OPA192IDBVR ERR2 buffer, U204 OPA820 LOx3, U205 OPA820 LOx3, U206 AD5696R, U30 OPA814DBVR, U31 OPA814DBVR, U45 AD835 demod, U46 AD835 demod

Commit message: Working towards a full set of pcbs in v7
Parts:
- U1: footprint Package_SO:MSOP-10-1EP_3x3mm_P0.5mm_EP2.2x3.1mm_Mask1.83x1.89mm_ThermalVias -> Package_SO:MSOP-10-1EP_3x3mm_P0.5mm_EP1.68x1.88mm
Changed lines of the file:
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@@
 			)
 		)
-		(property "Footprint" "Package_SO:MSOP-10-1EP_3x3mm_P0.5mm_EP2.2x3.1mm_Mask1.83x1.89mm_ThermalVias"
+		(property "Footprint" "Package_SO:MSOP-10-1EP_3x3mm_P0.5mm_EP1.68x1.88mm"
 			(at 196.596 58.674 0)
 			(hide yes)
