File: Laser_Driver_v7/DIG_Card/DIG_Card.kicad_sch (KiCad schematic)
At the start: 209 parts, among them J2 10MHz Ref SMA, J301 DIN41612_03x32_C_Split, J302 LO1 out SMA, J302B1 LO2 out SMA, U301 OPA192IDBVR MOD1 buffer, U302 OPA192IDBVR MOD2 buffer, U303 74LVC1G125 CLK10M bus buffer, U34 AD9833xRM, U35 AD9833xRM (ref), U38 AD9833xRM (ref), U39 AD9833xRM, U40 LMV7219M5, U41 SN74LVC1G3157DBVR, U42 CDCE913PWG4, U44 CR2013-MI2120, Y1 ASE-10.000MHZ-LC-T

Commit message: Working towards a full set of pcbs in v7
Parts:
- R104: value 50 -> 49R9 10MHz ref term
- VM_U23, VM_U25, VM_U26, VM_U27, VM_U28: value LM339 -> LM339B
Connections:
- net SPARE_CLK10M is gone; now on net CLK10M_BUS: R311.2
