File: Laser_Driver_v7/DIG_Card/DIG_Card.kicad_pcb (KiCad board)
At the start: 6 copper layers, 160 x 100 mm, 209 parts, among them J2 10MHz Ref SMA, J301 DIN41612_03x32_C_Split, J302 LO1 out SMA, J302B1 LO2 out SMA, U301 OPA192IDBVR MOD1 buffer, U302 OPA192IDBVR MOD2 buffer, U303 74LVC1G125 CLK10M bus buffer, U34 AD9833xRM, U35 AD9833xRM (ref), U38 AD9833xRM (ref), U39 AD9833xRM, U40 LMV7219M5, U41 SN74LVC1G3157DBVR, U42 CDCE913PWG4, U44 CR2013-MI2120, Y1 ASE-10.000MHZ-LC-T

Commit message: Working towards a full set of pcbs in v7
Parts:
- R104: value 50 -> 49R9 10MHz ref term
- VM_U23, VM_U25, VM_U26, VM_U27, VM_U28: value LM339 -> LM339B
- moved TP312 21.1 mm to (91.8, 75.7)
Connections:
- R311 pad 2: SPARE_CLK10M -> CLK10M_BUS
Routing:
- net CLK10M_BUS: track 0.00 -> 104.8 mm, vias 0 -> 3
- net SPARE_CLK10M: track 91.4 -> 0.00 mm, vias 1 -> 0
- net 3.3V: track 0.00 -> 49.5 mm
- net SCL_BUS: track 187.8 -> 212.6 mm
- net SDA_BUS: track 176.3 -> 198.9 mm
- net MOD2_BUS: track 151.9 -> 172.5 mm, vias 1 -> 3
- net -6V_TEC: track 53.1 -> 73.4 mm
- net +6V_TEC: track 57.4 -> 71.7 mm
- net ERR1_BUS: track 112.0 -> 123.0 mm
- net GND: track 32.6 -> 22.2 mm, vias 504 -> 503
- net 5Vref: track 51.0 -> 40.8 mm
- net +15V: track 206.9 -> 215.5 mm
- net ERR2_BUS: track 115.0 -> 123.4 mm
- net -5V: track 42.0 -> 50.3 mm
- net +5V_LASER: track 22.3 -> 30.6 mm
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
Commit message: minor updates and U for FBG
Other:
- board text added: "DIG_Card v7"
Changed lines of the file:
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@@
 	)
 	(embedded_fonts no)
+	(gr_text "DIG_Card v7"
+		(at 161.175 45.500 0)
+		(layer "B.SilkS")
+		(effects
+			(font
+				(size 1.5 1.5)
+				(thickness 0.25)
+			)
+			(justify mirror)
+		)
+	)
 )
