File: Laser_Driver_v7/pm22V/pm22V.kicad_sch (KiCad schematic)
At the start: 28 parts, among them J5 Screw_Terminal_01x03, J6 DIN41612_03x32_C_Split, Q1 IRF540NPBF, Q2 IRF9540NPBF

Commit message: Working towards a full set of pcbs in v7
Parts:
- D1: value GBPC1510-E4/51 -> GBPC1510W; symbol Diode_Bridge:GBU4M -> Diode_Bridge_GBPC:GBPC1510W; DigiKey P/N (none) -> 2616-GBPC1510W-ND; Manufacturer (none) -> Surge Components; Manufacturer Part Number (none) -> GBPC1510W
Other:
- note added: "DIN 41612 BACKPLANE CONNECTOR (Type C, 96-way, 3x32 @ 2.54 mm): Board: Harting 09031966921 (right-angle male, 96-way, THT). Mate: Harting 09032966855 (vertical female, backplane side). Contacts rated 2 A; the pinout is designed at 1.5 A derated, with every rail owning whole a/b/c columns. See SLOT_PINOUT_v7.md. This card drives +18V (col 7) and -18V (col 9); GND on cols 8 and 10. AC / transformer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"
- note removed: "DIN 41612 BACKPLANE CONNECTOR (Type H, 24 signal + 8 power): Board: TE/Erni 374144-E (right-angle male, 24+8, gold THT). Mate: TE/Erni 294711-E (vertical female, backplane side). 8 power blades ~10 A (+/-6V_TEC, +/-18V, returns); 24 signal ~2 A. AC / transformer leads stay on screw terminals J1-J5."
Changed lines of the file:
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@@
 		)
 	)
-	(text "DIN 41612 BACKPLANE CONNECTOR  (Type H, 24 signal + 8 power):\nBoard:  TE/Erni 374144-E  (right-angle male, 24+8, gold THT).\nMate:   TE/Erni 294711-E  (vertical female, backplane side).\n8 power blades ~10 A (+/-6V_TEC, +/-18V, returns); 24 signal ~2 A.\nAC / transformer leads stay on screw terminals J1-J5."
+	(text "DIN 41612 BACKPLANE CONNECTOR  (Type C, 96-way, 3x32 @ 2.54 mm):\nBoard:  Harting 09031966921  (right-angle male, 96-way, THT).\nMate:   Harting 09032966855  (vertical female, backplane side).\nContacts rated 2 A; the pinout is designed at 1.5 A derated, with every\nrail owning whole a/b/c columns.  See SLOT_PINOUT_v7.md.\nThis card drives +18V (col 7) and -18V (col 9); GND on cols 8 and 10.\nAC / transformer leads stay on screw terminal J5."
 		(exclude_from_sim no)
 		(at 21.59 122.174 0)
@@
 	)
 	(symbol
-		(lib_id "Diode_Bridge:GBU4M")
+		(lib_id "Diode_Bridge_GBPC:GBPC1510W")
 		(at 54.61 46.99 0)
 		(unit 1)
@@
 			)
 		)
-		(property "Value" "GBPC1510-E4/51"
+		(property "Value" "GBPC1510W"
 			(at 49.53 41.91 0)
 			(show_name no)
@@
 			)
 		)
-		(property "Datasheet" "http://www.vishay.com/docs/88656/gbu4a.pdf"
+		(property "Datasheet" "https://mm.digikey.com/Volume0/opasdata/d220001/medias/docus/3003/GBPC15.pdf"
 			(at 55.626 67.056 0)
 			(hide yes)
@@
 			)
 		)
-		(property "Description" "Single-Phase Bridge Rectifier, 700V Vrms, 4.0A If, GBU package"
+		(property "Description" "Single-Phase Bridge Rectifier, 1000 V, 15 A, GBPC-W package (wire leads)"
 			(at 55.88 64.516 0)
 			(hide yes)
 			(show_name no)
+			(do_not_autoplace no)
+			(effects
+				(font
+					(size 1.27 1.27)
+				)
+			)
+		)
+		(property "Manufacturer Part Number" "GBPC1510W"
+			(at 55.88 62 0)
+			(hide yes)
+			(show_name no)
+			(do_not_autoplace no)
+			(effects
+				(font
+					(size 1.27 1.27)
+				)
+			)
+		)
+		(property "Manufacturer" "Surge Components"
+			(at 55.88 62 0)
+			(hide yes)
+			(show_name no)
+			(do_not_autoplace no)
+			(effects
+				(font
+					(size 1.27 1.27)
+				)
+			)
+		)
+		(property "DigiKey P/N" "2616-GBPC1510W-ND"
+			(at 55.88 62 0)
+			(hide yes)
+			(show_name no)
