File: Laser_Driver_v7/pm22V/pm22V.kicad_pcb (KiCad board)
At the start: 2 copper layers, 160 x 100 mm, 28 parts, among them J5 Screw_Terminal_01x03, J6 DIN41612_03x32_C_Split, Q1 IRF540NPBF, Q2 IRF9540NPBF

Commit message: Working towards a full set of pcbs in v7
Parts:
- D1: value GBPC1510-E4/51 -> GBPC1510W
Changed lines of the file:
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@@
 			)
 		)
-		(property "Value" "GBPC1510-E4/51"
+		(property "Value" "GBPC1510W"
 			(at 9 -12.8 0)
 			(layer "F.Fab")
@@
 			)
 		)
-		(property "Datasheet" "http://www.vishay.com/docs/88656/gbu4a.pdf"
+		(property "Datasheet" "https://mm.digikey.com/Volume0/opasdata/d220001/medias/docus/3003/GBPC15.pdf"
 			(at 0 0 180)
 			(unlocked yes)
@@
 			)
 		)
-		(property "Description" "Single-Phase Bridge Rectifier, 700V Vrms, 4.0A If, GBU package"
+		(property "Description" "Single-Phase Bridge Rectifier, 1000 V, 15 A, GBPC-W package (wire leads)"
 			(at 0 0 180)
 			(unlocked yes)
@@
 			)
 		)
+		(property "Manufacturer Part Number" "GBPC1510W"
+			(at 0 0 0)
+			(unlocked yes)
+			(layer "F.Fab")
+			(hide yes)
+			(effects
+				(font
+					(size 1.27 1.27)
+					(thickness 0.15)
+				)
+			)
+		)
+		(property "Manufacturer" "Surge Components"
+			(at 0 0 0)
+			(unlocked yes)
+			(layer "F.Fab")
+			(hide yes)
+			(effects
+				(font
+					(size 1.27 1.27)
+					(thickness 0.15)
+				)
+			)
+		)
+		(property "DigiKey P/N" "2616-GBPC1510W-ND"
+			(at 0 0 0)
+			(unlocked yes)
+			(layer "F.Fab")
+			(hide yes)
+			(effects
+				(font
+					(size 1.27 1.27)
+					(thickness 0.15)
+				)
+			)
+		)
 		(property ki_fp_filters "Diode*Bridge*Vishay*GBU*")
 		(sheetname "/")
@@
 		)
 		(embedded_fonts no)
+			(model "C:/GIT/DualLaserPDHDriver/lib/Heatsinks.3dshapes/Boyd_6223BG.step"
+			(offset (xyz 0 0 7.3))
+			(scale (xyz 1 1 1))
+			(rotate (xyz 0 0 0))
+		)
 	)
 	(footprint "Capacitor_THT:CP_Radial_D16.0mm_P7.50mm"

Commit message: minor updates and U for FBG
Other:
- board text added: "pm22V v7"
Changed lines of the file:
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@@
 	)
 	(embedded_fonts no)
+	(gr_text "pm22V v7"
+		(at 116.100 50.250 0)
+		(layer "B.SilkS")
+		(effects
+			(font
+				(size 1.5 1.5)
+				(thickness 0.25)
+			)
+			(justify mirror)
+		)
+	)
 )
