File: Laser_Driver_v7/pm6V/pm6V.kicad_pcb (KiCad board)
At the start: 2 copper layers, 160 x 100 mm, 64 parts, among them J4 Screw_Terminal_01x03, J6 DIN41612_03x32_C_Split, Q10 Q_NPN MJL21194, Q3 IRF540ZPBF, Q4 IRF9540NPBF, Q5 MMBT2907, Q6 MMBT2222, Q7 Q_PNP_MJL21193, Q8 Q_PNP_MJL21193, Q9 Q_NPN MJL21194, U11 LM4051AIM3-ADJ/NOPB, U12 LM4051AIM3-ADJ/NOPB

Commit message: Working towards a full set of pcbs in v7
Parts:
- D7: value GBPC1510W-E4/51 -> GBPC1510W
- moved R39 15.9 mm to (75.6, 125.8), turned to 90 degrees
- moved C53 13.4 mm to (72.9, 125.8), turned to 90 degrees
- moved R38 2.80 mm to (68.9, 130.3)
- moved C52 2.80 mm to (72.0, 130.2)
Routing:
- net -6V_TEC: track 206.2 -> 197.0 mm
- net +6V_TEC: track 85.5 -> 79.4 mm, vias 13 -> 14
- net PGND_TEC: vias 166 -> 157
