File: Laser_Driver_v7/pm6V/pm6V.kicad_sch (KiCad schematic)
At the start: 64 parts, among them J4 Screw_Terminal_01x03, J6 DIN41612_03x32_C_Split, Q10 Q_NPN MJL21194, Q3 IRF540ZPBF, Q4 IRF9540NPBF, Q5 MMBT2907, Q6 MMBT2222, Q7 Q_PNP_MJL21193, Q8 Q_PNP_MJL21193, Q9 Q_NPN MJL21194, U11 LM4051AIM3-ADJ/NOPB, U12 LM4051AIM3-ADJ/NOPB

Commit message: Working towards a full set of pcbs in v7
Parts:
- D7: value GBPC1510W-E4/51 -> GBPC1510W; symbol Diode_Bridge:GBU4M -> Diode_Bridge_GBPC:GBPC1510W
Other:
- note added: "DIN 41612 BACKPLANE CONNECTOR (Type C, 96-way, 3x32 @ 2.54 mm): Board: Harting 09031966921 (right-angle male, 96-way, THT). Mate: Harting 09032966855 (vertical female, backplane side). Contacts rated 2 A; the pinout is designed at 1.5 A derated, with every rail owning whole a/b/c columns. See SLOT_PINOUT_v7.md. This card drives +6V_TEC (cols 1-2), PGND_TEC (cols 3-4) and -6V_TEC (cols 5-6): 6 con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"
- note added: "LM4051-ADJ (U11/U12) shunt ref: cathode to GND, anode toward base node"
- note added: "LM4051-ADJ set to 6.23 V by R24/R25 (60.4k/15k, Vref 1.24 V): sets base to +6.2 V; Vout = 6.2 - Vbe ~ +6.0 V"
- note added: "Pass devices (parallel pairs, emitter-ballasted): negative rail Q7/Q8 MJL21193 PNP via R34/R35 (0.1 R) positive rail Q9/Q10 MJL21194 NPN via R36/R37 (0.1 R) Raw from D7 off the +/-9 Vac secondary is about +/-11 V. (There is no Q17 on this board.)"
- note removed: "DIN 41612 BACKPLANE CONNECTOR (Type H, 24 signal + 8 power): Board: TE/Erni 374144-E (right-angle male, 24+8, gold THT). Mate: TE/Erni 294711-E (vertical female, backplane side). 8 power blades ~10 A (+/-6V_TEC, +/-22V, returns); 24 signal ~2 A. AC / transformer leads stay on screw terminals J1-J5."
- note removed: "LM4040-6.2: sets base to +6.2 V; Vout = 6.2 - Vbe ≈ +6.0 V"
- note removed: "LM4040: cathode to GND, anode toward base node"
- note removed: "Q17 MJL21193 PNP: emitter at raw -16.6 V; collector = -6 V output"
Changed lines of the file:
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@@
 		)
 	)
-	(text "LM4040: cathode to GND, anode toward base node"
+	(text "LM4051-ADJ (U11/U12) shunt ref: cathode to GND, anode toward base node"
 		(exclude_from_sim no)
 		(at 106.426 136.144 0)
@@
 		)
 	)
-	(text "DIN 41612 BACKPLANE CONNECTOR  (Type H, 24 signal + 8 power):\nBoard:  TE/Erni 374144-E  (right-angle male, 24+8, gold THT).\nMate:   TE/Erni 294711-E  (vertical female, backplane side).\n8 power blades ~10 A (+/-6V_TEC, +/-22V, returns); 24 signal ~2 A.\nAC / transformer leads stay on screw terminals J1-J5."
+	(text "DIN 41612 BACKPLANE CONNECTOR  (Type C, 96-way, 3x32 @ 2.54 mm):\nBoard:  Harting 09031966921  (right-angle male, 96-way, THT).\nMate:   Harting 09032966855  (vertical female, backplane side).\nContacts rated 2 A; the pinout is designed at 1.5 A derated, with every\nrail owning whole a/b/c columns.  See SLOT_PINOUT_v7.md.\nThis card drives +6V_TEC (cols 1-2), PGND_TEC (cols 3-4) and\n-6V_TEC (cols 5-6): 6 contacts each = 9 A derated, against the\n3 A/rail design point.\nAC / transformer leads stay on screw terminal J4."
 		(exclude_from_sim no)
 		(at 22.352 -13.716 0)
@@
 		)
 	)
-	(text "Q17 MJL21193 PNP: emitter at raw -16.6 V; collector = -6 V output"
+	(text "Pass devices (parallel pairs, emitter-ballasted):\n  negative rail  Q7/Q8   MJL21193 PNP   via R34/R35 (0.1 R)\n  positive rail  Q9/Q10  MJL21194 NPN   via R36/R37 (0.1 R)\nRaw from D7 off the +/-9 Vac secondary is about +/-11 V.\n(There is no Q17 on this board.)"
 		(exclude_from_sim no)
 		(at 104.648 133.858 0)
@@
 		)
 	)
-	(text "LM4040-6.2: sets base to +6.2 V; Vout = 6.2 - Vbe ≈ +6.0 V"
+	(text "LM4051-ADJ set to 6.23 V by R24/R25 (60.4k/15k, Vref 1.24 V):\nsets base to +6.2 V; Vout = 6.2 - Vbe ~ +6.0 V"
 		(exclude_from_sim no)
 		(at 87.122 89.916 0)
@@
 	)
 	(symbol
-		(lib_id "Diode_Bridge:GBU4M")
+		(lib_id "Diode_Bridge_GBPC:GBPC1510W")
 		(at 40.64 48.26 0)
 		(unit 1)
@@
 			)
 		)
-		(property "Value" "GBPC1510W-E4/51"
+		(property "Value" "GBPC1510W"
 			(at 28.956 44.704 0)
 			(show_name no)
