File: Laser_Driver_v7/CH_Card/CH_Card.kicad_sch (KiCad schematic)
At the start: 196 parts, among them J1 DIN41612_03x32_C_Split, Q13 IRL540N, Q14 IRF9540N, Q17 IRL540N, Q18 IRF9540N, Q19 DMN3404L, U101 AD5696R, U102 ADS1115, U103 PCA9538, U104 ADG419BRM, U105 ADG419BRM, U106 OPA192IDBVR, U107 OPA551U, U108 ADG419BRM, U17 OPA192IDBVR, U19 OPA192IDBVR, U21 OPA551U, U22 OPA192IDBVR, U24 OPA192IDBVR, U26 ADG419BRM, U28 INA828, U32 INA828

Commit message: Working on v7 docs and pcbs and 3d models
Parts:
- J_BTF1: value Butterfly harness header - Wurth WR-PHD 2x7 (mates LDM-BUTTERFLY) -> Butterfly daughter-card stacking header - Samtec TSW-107-21-G-D (30.99mm post)
Changed lines of the file:
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@@
 			)
 		)
-		(property "Value" "Butterfly harness header - Wurth WR-PHD 2x7 (mates LDM-BUTTERFLY)"
+		(property "Value" "Butterfly daughter-card stacking header - Samtec TSW-107-21-G-D (30.99mm post)"
 			(at 222.25 43.434 0)
 			(show_name no)
@@
 			)
 		)
-		(property "Datasheet" ""
+		(property "Datasheet" "https://suddendocs.samtec.com/catalog_english/tsw_th.pdf"
 			(at 222.25 29.21 0)
 			(hide yes)
@@
 			)
 		)
-		(property "Description" ""
+		(property "Description" "2x7 0.100in square-post header, lead style -21: 30.99mm mating post, 36.32mm OAL, pin tip 33.53mm above the board face. Carries the butterfly/DFB daughter card. Mates ESQ-107-12-G-D (11.05mm body, 2.29mm tail) at a 40mm board-to-board gap set by M3 x 40mm standoffs (Wurth 970400324 brass): insertion depth 4.58mm, Samtec spec 3.68-6.35mm. Standoffs set the gap and carry the daughter-card + heat-spreader mass - the pins are signal only. 5.2-6.3 A per pin."
 			(at 222.25 29.21 0)
 			(show_name no)

Commit message: Working towards a full set of pcbs in v7
Parts:
- removed H2: MountingHole, MountingHole:MountingHole_2.7mm, symbol Mechanical:MountingHole
- added C175: 10nF CASE shield RF bypass (par R75), Capacitor_SMD:C_0805_2012Metric_Pad1.18x1.45mm_HandSolder, symbol Device:C
- J_BTF1: footprint Connector_PinHeader_2.54mm:PinHeader_2x07_P2.54mm_Vertical -> Optical:BTF_Card_Mezzanine_2x07_M3
- R130: value 10k inv in -> 10k 0.1% inv in
- R131: value 10k inv fb -> 10k 0.1% inv fb
- R133: value 10k IMON fb -> 10k 0.1% IMON fb
- R_f1: value 10k Rf -> 10k 0.1% Rf
- R_f2: value 10k Rf TIA -> 10k 0.1% Rf TIA
Connections:
- net unconnected-(J_BTF1-NC-Pad12) is gone; now on net N_J_BTF1_CHIP_: J_BTF1.12 (NC)
- net unconnected-(J_BTF1-NC-Pad6) is gone; now on net GND: J_BTF1.6 (NC)
- net unconnected-(J_BTF1-NC-Pad7) is gone; now on net N_J_BTF1_NTC_A: J_BTF1.7 (NC)
- net unconnected-(J_BTF1-NC-Pad8) is gone; now on net N_J_BTF1_NTC_GND: J_BTF1.8 (NC)
- net unconnected-(J_BTF1-NC-Pad9) is gone; now on net N_J_BTF1_GND: J_BTF1.9 (NC)
- net GND: now also C175.2; no longer J_BTF1.3 (NC)
- net MPD_K: now also J_BTF1.5 (NTC_GND); no longer J_BTF1.4 (NC)
- net N_J_BTF1_CHIP_: no longer J_BTF1.11 (CHIP-)
- net N_J_BTF1_GND: now also J_BTF1.11 (CHIP-), J_BTF1.3 (NC), J_BTF1.4 (NC), C175.1; no longer J_BTF1.13 (GND)
- net N_J_BTF1_NTC_A: no longer J_BTF1.2 (NTC_A)
- net N_J_BTF1_NTC_GND: no longer J_BTF1.5 (NTC_GND)
- net N_J_BTF1_TECP: now also J_BTF1.2 (NTC_A)
- net N_J_BTF1_TEC_: now also J_BTF1.13 (GND)
- net N_J_BTF1_LD_A: now reaches J_BTF1.10 (CHIP+), R73.1

Commit message: Updates to capacitors for derating.
Parts:
- removed JP102: GA1 addr jumper, Connector_PinHeader_2.54mm:PinHeader_1x02_P2.54mm_Vertical, symbol CHCard_New:JP_ADDR
- removed JP103: GA2 addr jumper, Connector_PinHeader_2.54mm:PinHeader_1x02_P2.54mm_Vertical, symbol CHCard_New:JP_ADDR
- removed R128: 10k GA1 pullup, Resistor_SMD:R_0805_2012Metric_Pad1.20x1.40mm_HandSolder, symbol Device:R
- removed R129: 10k GA2 pullup, Resistor_SMD:R_0805_2012Metric_Pad1.20x1.40mm_HandSolder, symbol Device:R
- added C176: 100nF U105 +5V dec, Capacitor_SMD:C_0805_2012Metric_Pad1.18x1.45mm_HandSolder, symbol Device:C
- added C177: 100nF U108 +5V dec, Capacitor_SMD:C_0805_2012Metric_Pad1.18x1.45mm_HandSolder, symbol Device:C
- C76: value Ci 1n -> Ci 1n C0G
Connections:
- net GA1 is gone; now on net GND: U103.2 (A1)
- net GA2 is gone; now on net GND: U103.6 (IO2)
- net +5V: now also C176.1, C177.1
- net GND: now also C176.2, C177.2
Other:
- note added: "CARD ADDRESS via the SINGLE on-card jumper JP101 (10k pullup R127 to 3V3_DIG): FITTED = GA0 0 = ch1 card; OPEN = GA0 1 = ch2 card. One strap sets the I2C address AND the ERR/MOD bus pair, so there is nothing else to configure and no way to half-configure a card. v7: JP102/JP103 and pullups R128/R129 DELETED. GA1 was PCA9538 A1, and firmware fixes the expander at 0x70|GA0, so GA1 had exactly one l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"
- note removed: "CARD ADDRESS via on-card jumpers JP101-JP103 (10k pullups R127-R129 to 3V3_DIG): fit jumper = 0, open = 1."
