File: Laser_Driver_v7/pm1p8V_pm5V_5Vref_5Vlaser/pm1p8V_pm5V_5Vref_5Vlaser.kicad_sch (KiCad schematic)
At the start: 103 parts, among them J6 DIN41612_03x32_C_Split, U1 MC7808CTG, U10 LT3042EMSE +14.3V, U13 MC7812CTG, U14 MC7808CTG, U15 LT3045EMSE 5V, U16 LT3045EMSE 5V, U17 MC7808CTG, U18 MC7906CTG, U19 LT3045EMSE 5V, U2 LT3042EMSE +5.5V, U20 LT3094EMSE -5V, U21 OPA192IDBVR, U3 LTC6655BHMS8-5#PBF, U4 MC7812CTG, U5 MC7805CTG, U6 LT3045EMSE 3.3V, U7 LP5907MFX-1.8, U8 TPS7A3901DSCR, U9 LT3094EMSE -14.3V

Commit message: Working towards a full set of pcbs in v7
Connections:
- net 5Vref: now also J6.a20 (Pin_a20)
- net VREF_MID: now also J6.a22 (Pin_a22)
- no-connect marks 92 -> 87

Commit message: Updates to capacitors for derating.
Parts:
- added C34: 10uF 50V X7R, Capacitor_SMD:C_1210_3225Metric_Pad1.33x2.70mm_HandSolder, symbol Device:C
- added C35, C36, C37, C38: 100nF, Capacitor_SMD:C_0805_2012Metric_Pad1.18x1.45mm_HandSolder, symbol Device:C
- C13: value 4.7uF -> 10uF 25V X7R; footprint Capacitor_SMD:C_0805_2012Metric_Pad1.18x1.45mm_HandSolder -> Capacitor_SMD:C_1206_3216Metric_Pad1.33x1.80mm_HandSolder; DigiKey P/N 1276-2969-2-ND -> 399-C1206C106K3RACTUCT-ND; Manufacturer Samsung Electro-Mechanics -> KEMET; Manufacturer Part Number CL21B475KAFNNNE -> C1206C106K3RACTU
- C25, C26: value 10uF -> 4.7uF 50V X7R; DigiKey P/N 399-11939-2-ND -> 445-181404-1-ND; Manufacturer KEMET -> TDK; Manufacturer Part Number C0805C106K3PACTU -> CGA4J1X7R1H475K125AC
- C32, C33: value 10uF -> 10uF 50V X7R; footprint Capacitor_SMD:C_0805_2012Metric_Pad1.18x1.45mm_HandSolder -> Capacitor_SMD:C_1210_3225Metric_Pad1.33x2.70mm_HandSolder; DigiKey P/N 399-11939-2-ND -> 1276-3388-1-ND; Manufacturer KEMET -> Samsung Electro-Mechanics; Manufacturer Part Number C0805C106K3PACTU -> CL32B106KBJNNWE
- C54: value 4.7uF -> 4.7uF 50V X7R; DigiKey P/N 1276-2969-2-ND -> 445-181404-1-ND; Manufacturer Samsung Electro-Mechanics -> TDK; Manufacturer Part Number CL21B475KAFNNNE -> CGA4J1X7R1H475K125AC
- C61, C62, C71: value 10uF -> 22uF 25V X7R; footprint Capacitor_SMD:C_0805_2012Metric_Pad1.18x1.45mm_HandSolder -> Capacitor_SMD:C_1210_3225Metric_Pad1.33x2.70mm_HandSolder; DigiKey P/N 399-11939-2-ND -> 399-C1210C226M3RACTUCT-ND; Manufacturer Part Number C0805C106K3PACTU -> C1210C226M3RACTU
- C69: value 10uF X5R or X7R -> 22uF 25V X7R; footprint Capacitor_SMD:C_0805_2012Metric_Pad1.18x1.45mm_HandSolder -> Capacitor_SMD:C_1210_3225Metric_Pad1.33x2.70mm_HandSolder; DigiKey P/N 399-11939-2-ND -> 399-C1210C226M3RACTUCT-ND; Manufacturer Part Number C0805C106K3PACTU -> C1210C226M3RACTU
Connections:
- net +5V: now also C37.1
- net -15V: now also C34.2
- net -5V: now also C38.1
- net GND: now also C34.1, C35.2, C36.2, C37.2, C38.2
- net at C62.1, R43.1, U16.10 (OUTS)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: now also C36.1
- net at C61.1, R42.1, U15.10 (OUTS)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: now also C35.1
