File: Laser_Driver_v7/Backplane/Backplane_Slots.kicad_pcb (KiCad board)
At the start: 2 copper layers, 390.4 x 128.6 mm, 27 parts, among them J1 DIN41612_03x32_C_Split, J2 DIN41612_03x32_C_Split, J3 DIN41612_03x32_C_Split, J4 DIN41612_03x32_C_Split, J5 DIN41612_03x32_C_Split, J6 DIN41612_03x32_C_Split, J7 DIN41612_03x32_C_Split, J8 DIN41612_03x32_C_Split

Commit message: Working towards a full set of pcbs in v7
Parts:
- moved C1 22.8 mm to (404.4, 86.0)
- moved D3 22.8 mm to (407.8, 86.1)
- moved R1 22.8 mm to (402.1, 86.0)
Connections:
- net ERR1 renamed ERR1_BUS
- net ERR2 renamed ERR2_BUS
- net MOD1_DRV renamed MOD1_BUS
- net MOD2_DRV renamed MOD2_BUS
- net SCL renamed SCL_BUS
- net SDA renamed SDA_BUS
- net SPARE_CLK10M renamed CLK10M_BUS
Routing:
- net GND: track 4497.1 -> 3694.3 mm, vias 97 -> 10
- net -6V_TEC: track 0.00 -> 721.4 mm
- net ERR1_BUS: track 1031.6 -> 367.2 mm, vias 16 -> 0
- net PGND_TEC: track 1375.9 -> 721.4 mm, vias 56 -> 0
- net 3V3: track 930.5 -> 360.7 mm, vias 8 -> 0
- net -5V: track 814.5 -> 360.7 mm, vias 8 -> 0
- net SPARE_A31: track 0.00 -> 400.2 mm, vias 0 -> 7
- net SPARE_A32: track 0.00 -> 384.3 mm, vias 0 -> 7
- net SPARE_C32: track 0.00 -> 368.5 mm
- net 5Vref: track 0.00 -> 367.9 mm
- net CLK10M_BUS: track 0.00 -> 367.5 mm
- net ERR2_BUS: track 0.00 -> 367.5 mm
- net SCL_BUS: track 0.00 -> 367.4 mm
- net SPARE_C31: track 0.00 -> 367.3 mm
- net FAULT_n: track 0.00 -> 367.3 mm
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- added copper zone on B.Cu, net +15V
- added copper zone on F.Cu, net +15V
- added copper zone on B.Cu, net +18V
- added copper zone on F.Cu, net +18V
- added copper zone on B.Cu, net +5V
- added copper zone on F.Cu, net +5V
- added copper zone on B.Cu, net +5V_LASER
- added copper zone on F.Cu, net +5V_LASER
- added copper zone on B.Cu, net +6V_TEC
- added copper zone on F.Cu, net +6V_TEC
- added copper zone on B.Cu, net -15V
- added copper zone on F.Cu, net -15V
- added copper zone on B.Cu, net -18V
- added copper zone on F.Cu, net -18V
- added copper zone on B.Cu, net -5V
- added copper zone on F.Cu, net -5V
- added copper zone on B.Cu, net -6V_TEC
- added copper zone on F.Cu, net -6V_TEC
- added copper zone on B.Cu, net 1V8
- added copper zone on F.Cu, net 1V8
- added copper zone on B.Cu, net 3V3
- added copper zone on F.Cu, net 3V3

Commit message: minor updates and U for FBG
Other:
- board text added: "Backplane v7"
Changed lines of the file:
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@@
 	)
 	(embedded_fonts no)
+	(gr_text "Backplane v7"
+		(at 50.810 56.185 0)
+		(layer "B.SilkS")
+		(effects
+			(font
+				(size 1.5 1.5)
+				(thickness 0.25)
+			)
+			(justify mirror)
+		)
+	)
 )
