File: Laser_Driver_v7/BTF_Card/BTF_Card.kicad_pcb (KiCad board)
At the start: 2 copper layers, 43.4 x 75 mm, 9 parts, among them J1 ESQ-107-12-G-D

Commit message: Small changes for FBG option
Other:
- board text added: "BTF_Card v7"
Changed lines of the file:
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@@
 	)
 	(embedded_fonts no)
+	(gr_text "BTF_Card v7"
+		(at 92.425 37.100 0)
+		(layer "B.SilkS")
+		(effects
+			(font
+				(size 1.5 1.5)
+				(thickness 0.25)
+			)
+			(justify mirror)
+		)
+	)
 )
